Commit message: fixed another bug in URDF

File: mab_description/urdf/silver_badger.urdf.xacro (robot description, xacro)
@@ -88,4 +88,86 @@
   <link name="fr_l1">
     <inertial>
+      <origin rpy="0 0 0" xyz="0.031 -0.016 0"/>
+      <mass value="0.827"/>
+      <inertia ixx="0.0330" ixy="0" ixz="0" iyy="0.0077" iyz="0" izz="0.0286"/>
+    </inertial>
+    <visual>
+      <origin rpy="0 0 0" xyz="0 0 0"/>
+      <geometry>
+        <mesh filename="package://meshes/hb40/l1r.stl" scale="0.001 0.001 0.001"/>
+      </geometry>
+      <material name="orange"/>
+    </visual>
+    <collision>
+      <origin rpy="0 1.57 0" xyz="0.0 0 0"/>
+      <geometry>
+        <cylinder length="0.08" radius="0.05"/>
+      </geometry>
+    </collision>
+  </link>
+  <link name="fr_l2">
+    <inertial>
+      <origin rpy="0 0 0" xyz="0.001 -0.104 -0.003"/>
+      <mass value="0.118"/>
+      <inertia ixx="0.0213" ixy="0" ixz="0" iyy="0.0002" iyz="0" izz="0.0212"/>
+    </inertial>
+    <visual>
+      <origin rpy="0 0 0" xyz="0 0 0"/>
+      <geometry>
+        <mesh filename="package://meshes/hb40/l2r.stl" scale="0.001 0.001 0.001"/>
+      </geometry>
+      <material name="red"/>
+    </visual>
+    <collision>
+      <origin rpy="1.3 0 0" xyz="0 0.01 0.0055"/>
+      <geometry>
+        <cylinder length="0.0625" radius="0.01"/>
+      </geometry>
+      <material name="invisible"/>
+    </collision>
+    <collision>
+      <origin rpy="1.67 0.0 0.05" xyz="0 -0.1 0.005"/>
+      <geometry>
+        <cylinder length="0.2" radius="0.015"/>
+      </geometry>
+      <material name="invisible"/>
+    </collision>
+  </link>
+    <link name="fr_foot">
+    <inertial>
+      <origin rpy="0 0 0" xyz="0.0 0.0 0.0"/>
+      <mass value="0.0"/>
+      <inertia ixx="0.0" ixy="0" ixz="0" iyy="0.0" iyz="0" izz="0.0"/>
+    </inertial>
+    <visual>
+      <origin rpy="0 0 0" xyz="0 0 0"/>
+      <geometry>
+        <sphere radius="0.021"/>
+      </geometry>
+      <material name="black"/>
+    </visual>
+    <collision>
+      <origin rpy="0 0 0" xyz="0 0 0"/>
+      <geometry>
+        <sphere radius="0.02"/>
+      </geometry>
+    </collision>
+  </link>
+  <link name="fl_l0">
+    <inertial>
+      <origin rpy="0 0 0" xyz="0.0557 -0.016 0"/>
+      <mass value="0.645"/>
+      <inertia ixx="0.0052" ixy="0" ixz="0" iyy="0.0093" iyz="0" izz="0.0065"/>
+    </inertial>
+    <visual>
+      <origin rpy="0 0 0" xyz="0 0 0"/>
+      <geometry>
+        <mesh filename="package://meshes/hb40/l0l.stl" scale="0.001 0.001 0.001"/>
+      </geometry>
+      <material name="silver"/>
+    </visual>
+  </link>
+  <link name="fl_l1">
+    <inertial>
       <origin rpy="0 0 0" xyz="0.031 0.016 0"/>
       <mass value="0.827"/>
@@ -95,5 +177,5 @@
       <origin rpy="0 0 0" xyz="0 0 0"/>
       <geometry>
-        <mesh filename="package://meshes/hb40/l1r.stl" scale="0.001 0.001 0.001"/>
+        <mesh filename="package://meshes/hb40/l1lf.stl" scale="0.001 0.001 0.001"/>
       </geometry>
       <material name="orange"/>
@@ -106,7 +188,7 @@
     </collision>
   </link>
-  <link name="fr_l2">
-    <inertial>
-      <origin rpy="0 0 0" xyz="0.001 -0.104 -0.003"/>
+  <link name="fl_l2">
+    <inertial>
+      <origin rpy="0 0 0" xyz="0.001 0.104 -0.003"/>
       <mass value="0.118"/>
       <inertia ixx="0.0213" ixy="0" ixz="0" iyy="0.0002" iyz="0" izz="0.0212"/>
@@ -115,10 +197,10 @@
       <origin rpy="0 0 0" xyz="0 0 0"/>
       <geometry>
-        <mesh filename="package://meshes/hb40/l2r.stl" scale="0.001 0.001 0.001"/>
-      </geometry>
-      <material name="red"/>
-    </visual>
-    <collision>
-      <origin rpy="1.3 0 0" xyz="0 0.01 0.0055"/>
+        <mesh filename="package://meshes/hb40/l2l.stl" scale="0.001 0.001 0.001"/>
+      </geometry>
+      <material name="silver"/>
+    </visual>
+    <collision>
+      <origin rpy="-1.3 0.0 -0.00" xyz="0 -0.01 0.0055"/>
       <geometry>
         <cylinder length="0.0625" radius="0.01"/>
@@ -127,5 +209,5 @@
     </collision>
     <collision>
-      <origin rpy="1.67 0.0 0.05" xyz="0 -0.1 0.005"/>
+      <origin rpy="-1.67 0.0 -0.05" xyz="0 0.1 0.005"/>
       <geometry>
         <cylinder length="0.2" radius="0.015"/>
@@ -134,5 +216,5 @@
     </collision>
   </link>
-    <link name="fr_foot">
+  <link name="fl_foot">
     <inertial>
       <origin rpy="0 0 0" xyz="0.0 0.0 0.0"/>
@@ -154,5 +236,5 @@
     </collision>
   </link>
-  <link name="fl_l0">
+  <link name="rl_l0">
     <inertial>
       <origin rpy="0 0 0" xyz="0.0557 -0.016 0"/>
@@ -168,5 +250,5 @@
     </visual>
   </link>
-  <link name="fl_l1">
+  <link name="rl_l1">
     <inertial>
       <origin rpy="0 0 0" xyz="0.031 0.016 0"/>
@@ -188,5 +270,5 @@
     </collision>
   </link>
-  <link name="fl_l2">
+  <link name="rl_l2">
     <inertial>
       <origin rpy="0 0 0" xyz="0.001 0.104 -0.003"/>
@@ -202,5 +284,5 @@
     </visual>
     <collision>
-      <origin rpy="-1.3 0.0 -0.00" xyz="0 -0.01 0.0055"/>
+      <origin rpy="-1.3 0 0" xyz="0 -0.01 0.0055"/>
       <geometry>
         <cylinder length="0.0625" radius="0.01"/>
@@ -212,9 +294,9 @@
       <geometry>
         <cylinder length="0.2" radius="0.015"/>
-      </geometry>
-      <material name="invisible"/>
-    </collision>
-  </link>
-  <link name="fl_foot">
+        <material name="invisible"/>
+      </geometry>
+    </collision>
+  </link>
+  <link name="rl_foot">
     <inertial>
       <origin rpy="0 0 0" xyz="0.0 0.0 0.0"/>
@@ -236,5 +318,5 @@
     </collision>
   </link>
-  <link name="rl_l0">
+  <link name="rr_l0">
     <inertial>
       <origin rpy="0 0 0" xyz="0.0557 -0.016 0"/>
@@ -245,86 +327,4 @@
       <origin rpy="0 0 0" xyz="0 0 0"/>
       <geometry>
-        <mesh filename="package://meshes/hb40/l0l.stl" scale="0.001 0.001 0.001"/>
-      </geometry>
-      <material name="silver"/>
-    </visual>
-  </link>
-  <link name="rl_l1">
-    <inertial>
-      <origin rpy="0 0 0" xyz="0.031 0.016 0"/>
-      <mass value="0.827"/>
-      <inertia ixx="0.0330" ixy="0" ixz="0" iyy="0.0077" iyz="0" izz="0.0286"/>
-    </inertial>
-    <visual>
-      <origin rpy="0 0 0" xyz="0 0 0"/>
-      <geometry>
-        <mesh filename="package://meshes/hb40/l1lf.stl" scale="0.001 0.001 0.001"/>
-      </geometry>
-      <material name="orange"/>
-    </visual>
-    <collision>
-      <origin rpy="0 1.57 0" xyz="0.0 0 0"/>
-      <geometry>
-        <cylinder length="0.08" radius="0.05"/>
-      </geometry>
-    </collision>
-  </link>
-  <link name="rl_l2">
-    <inertial>
-      <origin rpy="0 0 0" xyz="0.001 0.104 -0.003"/>
-      <mass value="0.118"/>
-      <inertia ixx="0.0213" ixy="0" ixz="0" iyy="0.0002" iyz="0" izz="0.0212"/>
-    </inertial>
-    <visual>
-      <origin rpy="0 0 0" xyz="0 0 0"/>
-      <geometry>
-        <mesh filename="package://meshes/hb40/l2l.stl" scale="0.001 0.001 0.001"/>
-      </geometry>
-      <material name="silver"/>
-    </visual>
-    <collision>
-      <origin rpy="-1.3 0 0" xyz="0 -0.01 0.0055"/>
-      <geometry>
-        <cylinder length="0.0625" radius="0.01"/>
-      </geometry>
-      <material name="invisible"/>
-    </collision>
-    <collision>
-      <origin rpy="-1.67 0.0 -0.05" xyz="0 0.1 0.005"/>
-      <geometry>
-        <cylinder length="0.2" radius="0.015"/>
-        <material name="invisible"/>
-      </geometry>
-    </collision>
-  </link>
-  <link name="rl_foot">
-    <inertial>
-      <origin rpy="0 0 0" xyz="0.0 0.0 0.0"/>
-      <mass value="0.0"/>
-      <inertia ixx="0.0" ixy="0" ixz="0" iyy="0.0" iyz="0" izz="0.0"/>
-    </inertial>
-    <visual>
-      <origin rpy="0 0 0" xyz="0 0 0"/>
-      <geometry>
-        <sphere radius="0.021"/>
-      </geometry>
-      <material name="black"/>
-    </visual>
-    <collision>
-      <origin rpy="0 0 0" xyz="0 0 0"/>
-      <geometry>
-        <sphere radius="0.02"/>
-      </geometry>
-    </collision>
-  </link>
-  <link name="rr_l0">
-    <inertial>
-      <origin rpy="0 0 0" xyz="0.0557 -0.016 0"/>
-      <mass value="0.645"/>
-      <inertia ixx="0.0052" ixy="0" ixz="0" iyy="0.0093" iyz="0" izz="0.0065"/>
-    </inertial>
-    <visual>
-      <origin rpy="0 0 0" xyz="0 0 0"/>
-      <geometry>
         <mesh filename="package://meshes/hb40/l0r.stl" scale="0.001 0.001 0.001"/>
       </geometry>
@@ -334,5 +334,5 @@
   <link name="rr_l1">
     <inertial>
-      <origin rpy="0 0 0" xyz="0.031 0.016 0"/>
+      <origin rpy="0 0 0" xyz="0.031 -0.016 0"/>
       <mass value="0.827"/>
       <inertia ixx="0.0330" ixy="0" ixz="0" iyy="0.0077" iyz="0" izz="0.0286"/>
