Commit message: started adding ros_control but there is an error

File: mab_description/urdf/silver_badger.gazebo.xacro (robot description, xacro)
@@ -1,7 +1,5 @@
 <?xml version="1.0"?>
 <robot xmlns:xacro="http://www.ros.org/wiki/xacro">
-  <!-- Include materials-->
-  <!-- <xacro:include filename="$(find mab_description)/urdf/materials.xacro"/> -->
-  <!-- <xacro:macro name="silver_badger_gazebo"> -->
+    <!-- Colors-->
     <gazebo reference="base_link">
       <material>Gazebo/Grey</material>
@@ -61,4 +59,9 @@
       <material>Gazebo/Black</material>
     </gazebo>
-    <!-- </xacro:macro> -->
+    <!-- Controller-->
+    <gazebo>
+      <plugin name="gazebo_ros2_control" filename="libgazebo_ros2_control.so">
+        <parameters>$(find mab_gazebo)/config/silver_badger_controller.yaml</parameters>
+      </plugin>
+    </gazebo>
 </robot>

File: mab_description/urdf/silver_badger.urdf.xacro (robot description, xacro)
@@ -8,4 +8,55 @@
   <!-- Import Rviz colors -->
   <xacro:include filename="$(find mab_description)/urdf/materials.xacro" />
+  <!-- joint limits -->
+  <xacro:property name="fr_j0_limit_lower" value="-1.57"/>
+  <xacro:property name="fr_j0_limit_upper" value="1.57"/>
+  <xacro:property name="fr_j1_limit_lower" value="-1.57"/>
+  <xacro:property name="fr_j1_limit_upper" value="1.57"/>
+  <xacro:property name="fr_j2_limit_lower" value="-2.53"/>
+  <xacro:property name="fr_j2_limit_upper" value="0.0"/>
+  <xacro:property name="fl_j0_limit_lower" value="-1.57"/>
+  <xacro:property name="fl_j0_limit_upper" value="1.57"/>
+  <xacro:property name="fl_j1_limit_lower" value="-1.57"/>
+  <xacro:property name="fl_j1_limit_upper" value="1.57"/>
+  <xacro:property name="fl_j2_limit_lower" value="0.0"/>
+  <xacro:property name="fl_j2_limit_upper" value="2.53"/>
+  <xacro:property name="rl_j0_limit_lower" value="-1.57"/>
+  <xacro:property name="rl_j0_limit_upper" value="1.57"/>
+  <xacro:property name="rl_j1_limit_lower" value="-1.57"/>
+  <xacro:property name="rl_j1_limit_upper" value="1.57"/>
+  <xacro:property name="rl_j2_limit_lower" value="0.0"/>
+  <xacro:property name="rl_j2_limit_upper" value="2.53"/>
+  <xacro:property name="rr_j0_limit_lower" value="-1.57"/>
+  <xacro:property name="rr_j0_limit_upper" value="1.57"/>
+  <xacro:property name="rr_j1_limit_lower" value="-1.57"/>
+  <xacro:property name="rr_j1_limit_upper" value="1.57"/>
+  <xacro:property name="rr_j2_limit_lower" value="-2.53"/>
+  <xacro:property name="rr_j2_limit_upper" value="0.0"/>
+  <!-- max torques per joint -->
+  <xacro:property name="fr_j0_max_effort" value="16"/>
+  <xacro:property name="fr_j1_max_effort" value="16"/>
+  <xacro:property name="fr_j2_max_effort" value="16"/>
+  <xacro:property name="fl_j0_max_effort" value="16"/>
+  <xacro:property name="fl_j1_max_effort" value="16"/>
+  <xacro:property name="fl_j2_max_effort" value="16"/>
+  <xacro:property name="rl_j0_max_effort" value="16"/>
+  <xacro:property name="rl_j1_max_effort" value="16"/>
+  <xacro:property name="rl_j2_max_effort" value="16"/>
+  <xacro:property name="rr_j0_max_effort" value="16"/>
+  <xacro:property name="rr_j1_max_effort" value="16"/>
+  <xacro:property name="rr_j2_max_effort" value="16"/>
+  <!-- max velocities per joint -->
+  <xacro:property name="fr_j0_max_velocity" value="25"/>
+  <xacro:property name="fr_j1_max_velocity" value="25"/>
+  <xacro:property name="fr_j2_max_velocity" value="25"/>
+  <xacro:property name="fl_j0_max_velocity" value="25"/>
+  <xacro:property name="fl_j1_max_velocity" value="25"/>
+  <xacro:property name="fl_j2_max_velocity" value="25"/>
+  <xacro:property name="rl_j0_max_velocity" value="25"/>
+  <xacro:property name="rl_j1_max_velocity" value="25"/>
+  <xacro:property name="rl_j2_max_velocity" value="25"/>
+  <xacro:property name="rr_j0_max_velocity" value="25"/>
+  <xacro:property name="rr_j1_max_velocity" value="25"/>
+  <xacro:property name="rr_j2_max_velocity" value="25"/>
   <!--
   ##########################################################
@@ -405,4 +456,5 @@
   ##########################################################
   -->
+  <!-- Front Right Leg -->
   <joint armature="0.01" name="fr_j0" type="continuous">
     <parent link="body"/>
@@ -410,5 +462,5 @@
     <origin rpy="0 0 0" xyz="0.1375 -0.064 0"/>
     <axis xyz="1.0 0 0"/>
-    <limit effort="16.0" lower="-1.57" upper="1.57" velocity="25.0"/>
+    <limit effort="${fr_j0_max_effort}" lower="${fr_j0_limit_lower}" upper="${fr_j0_limit_upper}" velocity="${fr_j0_max_velocity}"/>
   </joint>
   <joint name="fr_j1" type="continuous">
@@ -417,5 +469,5 @@
     <origin rpy="0 0 -1.57" xyz="0.0555 -0.0125 0"/>
     <axis xyz="1.0 0 0"/>
-    <limit effort="16.0" lower="-1.57" upper="1.57" velocity="25.0"/>
+    <limit effort="${fr_j1_max_effort}" lower="${fr_j1_limit_lower}" upper="${fr_j1_limit_upper}" velocity="${fr_j1_max_velocity}"/>
   </joint>
   <joint name="fr_j2" type="continuous">
@@ -424,5 +476,5 @@
     <origin rpy="2.909 0 0" xyz="0.0584 -0.200 0"/>
     <axis xyz="1.0 0 0"/>
-    <limit effort="16.0" lower="-2.53" upper="0.0" velocity="25.0"/>
+    <limit effort="${fr_j2_max_effort}" lower="${fr_j2_limit_lower}" upper="${fr_j2_limit_upper}" velocity="${fr_j2_max_velocity}"/>
   </joint>
   <joint name="fr_jFoot" type="fixed">
@@ -432,4 +484,5 @@
     <axis xyz="0.0 0 0"/>
   </joint>
+  <!-- Front Left Leg -->
   <joint armature="0.01" name="fl_j0" type="continuous">
     <parent link="body"/>
@@ -437,5 +490,5 @@
     <origin rpy="0 0 0" xyz="0.1375 0.064 0"/>
     <axis xyz="1.0 0 0"/>
-    <limit effort="16.0" lower="-1.57" upper="1.57" velocity="25.0"/>
+    <limit effort="${fl_j0_max_effort}" lower="${fl_j0_limit_lower}" upper="${fl_j0_limit_upper}" velocity="${fl_j0_max_velocity}"/>
   </joint>
   <joint name="fl_j1" type="continuous">
@@ -444,5 +497,5 @@
     <origin rpy="0 0 1.57" xyz="0.0555 0.0125 0"/>
     <axis xyz="1.0 0 0"/>
-    <limit effort="16.0" lower="-1.57" upper="1.57" velocity="25.0"/>
+    <limit effort="${fl_j1_max_effort}" lower="${fl_j1_limit_lower}" upper="${fl_j1_limit_upper}" velocity="${fl_j1_max_velocity}"/>
   </joint>
   <joint name="fl_j2" type="continuous">
@@ -451,5 +504,5 @@
     <origin rpy="-2.909 0 0" xyz="0.0584 0.200 0"/>
     <axis xyz="1.0 0 0"/>
-    <limit effort="16.0" lower="0" upper="2.53" velocity="25.0"/>
+    <limit effort="${fl_j2_max_effort}" lower="${fl_j2_limit_lower}" upper="${fl_j2_limit_upper}" velocity="${fl_j2_max_velocity}"/>
   </joint>
   <joint name="fl_jFoot" type="fixed">
@@ -459,4 +512,5 @@
     <axis xyz="0.0 0 0"/>
   </joint>
+  <!-- Rear Left Leg -->
   <joint armature="0.01" name="rl_j0" type="continuous">
     <parent link="rear"/>
@@ -464,5 +518,5 @@
     <origin rpy="0 0 1.57" xyz="-0.1025 0.10765 0"/>
     <axis xyz="1.0 0 0"/>
-    <limit effort="16.0" lower="-1.57" upper="1.57" velocity="25.0"/>
+    <limit effort="${rl_j0_max_effort}" lower="${rl_j0_limit_lower}" upper="${rl_j0_limit_upper}" velocity="${rl_j0_max_velocity}"/>
   </joint>
   <joint name="rl_j1" type="continuous">
@@ -471,5 +525,5 @@
     <origin rpy="3.14159 0 1.57" xyz="0.0555 0.0125 0"/>
     <axis xyz="1.0 0 0"/>
-    <limit effort="16.0" lower="-1.57" upper="1.57" velocity="25.0"/>
+    <limit effort="${rl_j1_max_effort}" lower="${rl_j1_limit_lower}" upper="${rl_j1_limit_upper}" velocity="${rl_j1_max_velocity}"/>
   </joint>
   <joint name="rl_j2" type="continuous">
@@ -478,5 +532,5 @@
     <origin rpy="-2.909 0 0" xyz="0.0584 0.20 0"/>
     <axis xyz="1.0 0 0"/>
-    <limit effort="16.0" lower="0" upper="2.53" velocity="25.0"/>
+    <limit effort="${rl_j2_max_effort}" lower="${rl_j2_limit_lower}" upper="${rl_j2_limit_upper}" velocity="${rl_j2_max_velocity}"/>
   </joint>
   <joint name="rl_jFoot" type="fixed">
@@ -486,4 +540,5 @@
     <axis xyz="0.0 0 0"/>
   </joint>
+  <!-- Rear Right Leg -->
   <joint armature="0.01" name="rr_j0" type="continuous">
     <parent link="rear"/>
@@ -491,5 +546,5 @@
     <origin rpy="0 0 1.57" xyz="0.0255 0.10725 0"/>
     <axis xyz="1.0 0 0"/>
-    <limit effort="16.0" lower="-1.57" upper="1.57" velocity="25.0"/>
+    <limit effort="${rr_j0_max_effort}" lower="${rr_j0_limit_lower}" upper="${rr_j0_limit_upper}" velocity="${rr_j0_max_velocity}"/>
   </joint>
   <joint name="rr_j1" type="continuous">
@@ -498,5 +553,5 @@
     <origin rpy="3.14159 0 -1.57" xyz="0.0555 -0.0125 0"/>
     <axis xyz="1.0 0 0"/>
-    <limit effort="16.0" lower="-1.57" upper="1.57" velocity="25.0"/>
+    <limit effort="${rr_j1_max_effort}" lower="${rr_j1_limit_lower}" upper="${rr_j1_limit_upper}" velocity="${rr_j1_max_velocity}"/>
   </joint>
   <joint name="rr_j2" type="continuous">
@@ -505,5 +560,5 @@
     <origin rpy="2.909 0 0" xyz="0.0584 -0.20 0"/>
     <axis xyz="1.0 0 0"/>
-    <limit effort="16.0" lower="-2.53" upper="0.0" velocity="25.0"/>
+    <limit effort="${rr_j2_max_effort}" lower="${rr_j2_limit_lower}" upper="${rr_j2_limit_upper}" velocity="${rr_j2_max_velocity}"/>
   </joint>
   <joint name="rr_jFoot" type="fixed">
