Commit message: urdf loads in gazebo -- errors fixed in urdf

File: mab_description/urdf/silver_badger.urdf (robot description, URDF)
Before this commit: robot intention, 19 links, 18 joints
Links:
- link body: geometry collision box size=0.22 0.2 0.1; visual mesh filename=package://meshes/hb40/body.stl scale=0.001 0.001 0.001
- link fl_l0: geometry visual mesh filename=package://meshes/hb40/l0l.stl scale=0.001 0.001 0.001
- link fl_l1: geometry collision cylinder length=0.08 radius=0.05; visual mesh filename=package://meshes/hb40/l1lf.stl scale=0.001 0.001 0.001
- link fl_l2: geometry collision cylinder length=0.0625 radius=0.01; collision cylinder length=0.2 radius=0.015
- link fr_l0: geometry visual mesh filename=package://meshes/hb40/l0r.stl scale=0.001 0.001 0.001
- link fr_l1: geometry collision cylinder length=0.08 radius=0.05; visual mesh filename=package://meshes/hb40/l1r.stl scale=0.001 0.001 0.001
- link fr_l2: geometry collision cylinder length=0.0625 radius=0.01; collision cylinder length=0.2 radius=0.015
- link rear: geometry collision box size=0.2 0.05 0.1; visual mesh filename=package://meshes/hb40/rear.stl scale=0.001 0.001 0.001
- link rl_l0: geometry visual mesh filename=package://meshes/hb40/l0l.stl scale=0.001 0.001 0.001
- link rl_l1: geometry collision cylinder length=0.08 radius=0.05; visual mesh filename=package://meshes/hb40/l1lf.stl scale=0.001 0.001 0.001
- link rl_l2: geometry collision cylinder length=0.0625 radius=0.01; collision cylinder length=0.2 radius=0.015
- link rr_l0: geometry visual mesh filename=package://meshes/hb40/l0r.stl scale=0.001 0.001 0.001
- link rr_l1: geometry collision cylinder length=0.08 radius=0.05; visual mesh filename=package://meshes/hb40/l1r.stl scale=0.001 0.001 0.001
- link rr_l2: geometry collision cylinder length=0.0625 radius=0.01; collision cylinder length=0.2 radius=0.015

File: mab_description/urdf/silver_badger_rviz.urdf (robot description, URDF)
Before this commit: robot intention, 19 links, 18 joints
Links:
- link body: geometry collision box size=0.22 0.2 0.1; visual mesh filename=package://mab_description/meshes/hb40/body.stl scale=0.001 0.001 0.001
- link fl_l0: geometry visual mesh filename=package://mab_description/meshes/hb40/l0l.stl scale=0.001 0.001 0.001
- link fl_l1: geometry collision cylinder length=0.08 radius=0.05; visual mesh filename=package://mab_description/meshes/hb40/l1lf.stl scale=0.001 0.001 0.001
- link fl_l2: geometry collision cylinder length=0.0625 radius=0.01; collision cylinder length=0.2 radius=0.015
- link fr_l0: geometry visual mesh filename=package://mab_description/meshes/hb40/l0r.stl scale=0.001 0.001 0.001
- link fr_l1: geometry collision cylinder length=0.08 radius=0.05; visual mesh filename=package://mab_description/meshes/hb40/l1r.stl scale=0.001 0.001 0.001
- link fr_l2: geometry collision cylinder length=0.0625 radius=0.01; collision cylinder length=0.2 radius=0.015
- link rear: geometry collision box size=0.2 0.05 0.1; visual mesh filename=package://mab_description/meshes/hb40/rear.stl scale=0.001 0.001 0.001
- link rl_l0: geometry visual mesh filename=package://mab_description/meshes/hb40/l0l.stl scale=0.001 0.001 0.001
- link rl_l1: geometry collision cylinder length=0.08 radius=0.05; visual mesh filename=package://mab_description/meshes/hb40/l1lf.stl scale=0.001 0.001 0.001
- link rl_l2: geometry collision cylinder length=0.0625 radius=0.01; collision cylinder length=0.2 radius=0.015
- link rr_l0: geometry visual mesh filename=package://mab_description/meshes/hb40/l0r.stl scale=0.001 0.001 0.001
- link rr_l1: geometry collision cylinder length=0.08 radius=0.05; visual mesh filename=package://mab_description/meshes/hb40/l1r.stl scale=0.001 0.001 0.001
- link rr_l2: geometry collision cylinder length=0.0625 radius=0.01; collision cylinder length=0.2 radius=0.015
