Commit message: progress with slam

File: mab_description/urdf/silver_badger.urdf (robot description, URDF)
Before this commit: robot silver_badger, 19 links, 18 joints
Links:
- added link camera_interface, mass 0; visual mesh filename=package://meshes/camera_mount/camera-interface-realsense-an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 scale=0.001 0.001 0.001
- added link camera_mount, mass 0; visual mesh filename=package://meshes/camera_mount/hb-camera-mount.stl
- added link d435_camera__bottom_screw_frame
- added link d435_camera__color_frame
- added link d435_camera__color_optical_frame
- added link d435_camera__depth_frame
- added link d435_camera__depth_optical_frame
- added link d435_camera__infra1_frame
- added link d435_camera__infra1_optical_frame
- added link d435_camera__infra2_frame
- added link d435_camera__infra2_optical_frame
- added link d435_camera__link, mass 0.072; collision box size=0.02505 0.09 0.025; visual mesh filename=file:///home/aditya/ros2_ws/install/realsense2_description/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
- added link d435_camera__usb_plug_link; collision mesh filename=file:///home/aditya/ros2_ws/install/realsense2_description/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; visual mesh filename=file:///home/aditya/ros2_ws/install/realsense2_description/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
- added link imu_link, mass 0.0; visual box size=0.01 0.01 0.01
Joints:
- added joint camera_interface_joint: type fixed, parent body, child camera_interface
- added joint camera_mount_joint: type fixed, parent body, child camera_mount
- added joint d435_camera__color_joint: type fixed, parent d435_camera__link, child d435_camera__color_frame, origin xyz=0 0.015 0 rpy=0 0 0
- added joint d435_camera__color_optical_joint: type fixed, parent d435_camera__color_frame, child d435_camera__color_optical_frame, origin xyz=0 0 0 rpy=-1.5707963267948966 0 -1.5707963267948966
- added joint d435_camera__depth_joint: type fixed, parent d435_camera__link, child d435_camera__depth_frame, origin xyz=0 0 0 rpy=0 0 0
- added joint d435_camera__depth_optical_joint: type fixed, parent d435_camera__depth_frame, child d435_camera__depth_optical_frame, origin xyz=0 0 0 rpy=-1.5707963267948966 0 -1.5707963267948966
- added joint d435_camera__infra1_joint: type fixed, parent d435_camera__link, child d435_camera__infra1_frame, origin xyz=0 0.0 0 rpy=0 0 0
- added joint d435_camera__infra1_optical_joint: type fixed, parent d435_camera__infra1_frame, child d435_camera__infra1_optical_frame, origin xyz=0 0 0 rpy=-1.5707963267948966 0 -1.5707963267948966
- added joint d435_camera__infra2_joint: type fixed, parent d435_camera__link, child d435_camera__infra2_frame, origin xyz=0 -0.05 0 rpy=0 0 0
- added joint d435_camera__infra2_optical_joint: type fixed, parent d435_camera__infra2_frame, child d435_camera__infra2_optical_frame, origin xyz=0 0 0 rpy=-1.5707963267948966 0 -1.5707963267948966
- added joint d435_camera__joint: type fixed, parent camera_interface, child d435_camera__bottom_screw_frame, origin xyz=0.275855 -0.012447000000000001 0.068583 rpy=-1.5707963267948966 0 0
- added joint d435_camera__link_joint: type fixed, parent d435_camera__bottom_screw_frame, child d435_camera__link, origin xyz=0.010600000000000002 0.0175 0.0125 rpy=0 0 0
- added joint d435_camera__usb_plug_joint: type fixed, parent d435_camera__link, child d435_camera__usb_plug_link, origin xyz=-0.00605 -0.0528 0 rpy=0 0 0
- added joint imu_joint: type fixed, parent body, child imu_link

File: mab_description/xacro/camera.xacro (robot description, xacro)
@@ -2,22 +2,185 @@
 <robot name="realsense2_camera" xmlns:xacro="http://ros.org/wiki/xacro">
     <xacro:macro name="realsense2_camera" params="parent name">
+        <xacro:property name="M_PI" value="3.1415926535897931" />
+        <!-- The following values model the aluminum peripherial case for the
+        D435 camera, with the camera joint represented by the actual
+        peripherial camera tripod mount -->
+        <xacro:property name="d435_cam_height" value="0.025"/>
+        <xacro:property name="d435_cam_depth" value="0.02505"/>
+        <xacro:property name="d435_cam_mount_from_center_offset" value="0.0149"/>
+        <!-- glass cover is 0.1 mm inwards from front aluminium plate -->
+        <xacro:property name="d435_glass_to_front" value="0.1e-3"/>
+        <!-- see datasheet Revision 007, Fig. 4-4 page 65 -->
+        <xacro:property name="d435_zero_depth_to_glass" value="4.2e-3"/>
+        <!-- convenience precomputation to avoid clutter-->
+        <xacro:property name="d435_mesh_x_offset" value="${d435_cam_mount_from_center_offset-d435_glass_to_front-d435_zero_depth_to_glass}"/>
+        <xacro:property name="d435_cam_depth_px" value="${d435_cam_mount_from_center_offset}"/>
+        <xacro:property name="d435_cam_depth_py" value="0.0175"/>
+        <xacro:property name="d435_cam_depth_pz" value="${d435_cam_height/2}"/>
+        <!-- Camera position in 3D-->
+        <xacro:property name="d435_cam_x" value="0.290755"/>
+        <xacro:property name="d435_cam_y" value="0.000053"/>
+        <xacro:property name="d435_cam_z" value="0.068583"/>
+        <xacro:property name="d435_cam_roll" value="${-M_PI/2}"/>
         <!-- Initialize camera-->
         <xacro:include filename="$(find realsense2_description)/urdf/_d435.urdf.xacro"/>
-        <xacro:sensor_d435 parent="base_link" name="${name}">
-        <origin xyz="0 0 0.5" rpy="0 0 0"/>
+        <xacro:sensor_d435 parent="${parent}" name="${name}" use_nominal_extrinsics="false">
+            <origin xyz="${0.290755-d435_mesh_x_offset-d435_zero_depth_to_glass - d435_glass_to_front} ${0.000053-d435_cam_depth_pz} ${0.068583}" rpy="${-M_PI/2} 0 0"/>
         </xacro:sensor_d435>
-        <!-- Include the RealSense Camera Gazebo Macro -->
-        <xacro:include filename="$(find realsense2_description)/urdf/_d435.gazebo.xacro"/>
-        <!-- Use the RealSense Camera Gazebo Macro -->
-        <xacro:gazebo_d435
-        camera_name="${name}"
-        reference_link="${name}_link"
-        topics_ns="/${name}"
-        depth_optical_frame="${name}_depth_optical_frame"
-        color_optical_frame="${name}_color_optical_frame"
-        infrared1_optical_frame="${name}_infrared1_optical_frame"
-        infrared2_optical_frame="${name}_infrared2_optical_frame"
-        publish_pointcloud="true">
-        </xacro:gazebo_d435>
+        <!-- Link for camera image and gazebe plugin-->
+        <link name="camera_image_link">
+            <inertial>
+                <origin xyz="0 0 0" />
+                <mass value="0" />
+                <inertia ixx="0" ixy="0" ixz="0" iyy="0" iyz="0" izz="0" />
+            </inertial>
+            <visual>
+                <origin rpy="${d435_cam_roll} 0 0" xyz="${d435_cam_x} ${d435_cam_y} ${d435_cam_z}" />
+            </visual>
+        </link>
+        <joint name="camera_image_joint" type="fixed">
+            <parent link="${parent}"/>
+            <child link="camera_image_link"/>
+            <origin rpy="${d435_cam_roll} 0 0" xyz="${d435_cam_x} ${d435_cam_y} ${d435_cam_z}" />
+        </joint>
+        <!-- Some parameters-->
+        <xacro:property name="camera_name" value="${name}" />
+        <xacro:property name="topics_ns" value="/${name}" />
+        <xacro:property name="depth_optical_frame" value="${name}_depth_optical_frame" />
+        <xacro:property name="color_optical_frame" value="${name}_color_optical_frame" />
+        <xacro:property name="infrared1_optical_frame" value="${name}_infra1_frame" />
+        <xacro:property name="infrared2_optical_frame" value="${name}_infra2_frame" />
+        <xacro:property name="publish_pointcloud" value="true" />
+        <!-- Gazebo stuff for realsense-->
+        <!-- Load parameters to model's main link-->
+        <xacro:property name="deg_to_rad" value="0.01745329251994329577" />
+        <gazebo reference="camera_image_link">
+            <self_collide>0</self_collide>
+            <enable_wind>0</enable_wind>
+            <kinematic>0</kinematic>
+            <gravity>1</gravity>
+            <!--<mu>1</mu>-->
+            <mu2>1</mu2>
+            <fdir1>0 0 0</fdir1>
+            <!--<slip1>0</slip1>
+            <slip2>0</slip2>-->
+            <kp>1e+13</kp>
+            <kd>1</kd>
+            <!--<max_vel>0.01</max_vel>
+            <min_depth>0</min_depth>-->
+            <sensor name="${camera_name}color" type="camera">
+                <camera name="${camera_name}">
+                    <horizontal_fov>${69.4*deg_to_rad}</horizontal_fov>
+                    <image>
+                        <width>640</width>
+                        <height>480</height>
+                        <format>RGB_INT8</format>
+                    </image>
+                    <clip>
+                        <near>0.1</near>
+                        <far>100</far>
+                    </clip>
+                    <noise>
+                        <type>gaussian</type>
+                        <mean>0.0</mean>
+                        <stddev>0.007</stddev>
+                    </noise>
+                </camera>
+                <always_on>1</always_on>
+                <update_rate>30</update_rate>
+                <visualize>1</visualize>
+            </sensor>
+            <sensor name="${camera_name}ired1" type="camera">
+                <camera name="${camera_name}">
+                    <horizontal_fov>${85.2*deg_to_rad}</horizontal_fov>
+                    <image>
+                        <width>1280</width>
+                        <height>720</height>
+                        <format>L_INT8</format>
+                    </image>
+                    <clip>
+                        <near>0.1</near>
+                        <far>100</far>
+                    </clip>
+                    <noise>
+                        <type>gaussian</type>
+                        <mean>0.0</mean>
+                        <stddev>0.05</stddev>
+                    </noise>
+                </camera>
+                <always_on>1</always_on>
+                <update_rate>90</update_rate>
+                <visualize>0</visualize>
+            </sensor>
+            <sensor name="${camera_name}ired2" type="camera">
+                <camera name="${camera_name}">
+                    <horizontal_fov>${85.2*deg_to_rad}</horizontal_fov>
+                    <image>
+                        <width>1280</width>
+                        <height>720</height>
+                        <format>L_INT8</format>
+                    </image>
+                    <clip>
+                        <near>0.1</near>
+                        <far>100</far>
+                    </clip>
+                    <noise>
+                        <type>gaussian</type>
+                        <mean>0.0</mean>
+                        <stddev>0.05</stddev>
+                    </noise>
+                </camera>
+                <always_on>1</always_on>
+                <update_rate>90</update_rate>
+                <visualize>0</visualize>
+            </sensor>
+            <sensor name="${camera_name}depth" type="depth">
+                <camera name="${camera_name}">
+                    <horizontal_fov>${85.2*deg_to_rad}</horizontal_fov>
+                    <image>
+                        <width>1280</width>
+                        <height>720</height>
+                    </image>
+                    <clip>
+                        <near>0.1</near>
+                        <far>100</far>
+                    </clip>
+                    <noise>
+                        <type>gaussian</type>
+                        <mean>0.0</mean>
+                        <stddev>0.100</stddev>
+                    </noise>
+                </camera>
+                <always_on>1</always_on>
+                <update_rate>90</update_rate>
+                <visualize>0</visualize>
+            </sensor>
+        </gazebo>
+        <gazebo>
+            <plugin name="${topics_ns}" filename="librealsense_gazebo_plugin.so">
+                <prefix>${camera_name}</prefix>
+                <depthUpdateRate>30.0</depthUpdateRate>
+                <colorUpdateRate>30.0</colorUpdateRate>
+                <infraredUpdateRate>30.0</infraredUpdateRate>
+                <depthTopicName>${topics_ns}/depth/image_raw</depthTopicName>
+                <depthCameraInfoTopicName>${topics_ns}/depth/camera_info</depthCameraInfoTopicName>
+                <colorTopicName>${topics_ns}/color/image_raw</colorTopicName>
+                <colorCameraInfoTopicName>${topics_ns}/color/camera_info</colorCameraInfoTopicName>
+                <infrared1TopicName>${topics_ns}/infra1/image_raw</infrared1TopicName>
+                <infrared1CameraInfoTopicName>${topics_ns}/infra1/camera_info</infrared1CameraInfoTopicName>
+                <infrared2TopicName>${topics_ns}/infra2/image_raw</infrared2TopicName>
+                <infrared2CameraInfoTopicName>${topics_ns}/infra2/camera_info</infrared2CameraInfoTopicName>
+                <colorOpticalframeName>${color_optical_frame}</colorOpticalframeName>
+                <depthOpticalframeName>${depth_optical_frame}</depthOpticalframeName>
+                <infrared1OpticalframeName>${infrared1_optical_frame}</infrared1OpticalframeName>
+                <infrared2OpticalframeName>${infrared2_optical_frame}</infrared2OpticalframeName>
+                <rangeMinDepth>0.2</rangeMinDepth>
+                <rangeMaxDepth>10.0</rangeMaxDepth>
+                <pointCloud>${publish_pointcloud}</pointCloud>
+                <pointCloudTopicName>${topics_ns}/depth/color/points</pointCloudTopicName>
+                <pointCloudCutoff>0.25</pointCloudCutoff>
+                <pointCloudCutoffMax>9.0</pointCloudCutoffMax>
+            </plugin>
+        </gazebo>
         <!-- Adjust color for gazebo-->
         <gazebo reference="${name}_link">

File: mab_description/xacro/silver_badger.gazebo.xacro (robot description, xacro)
@@ -104,4 +104,10 @@
       <material>Gazebo/Black</material>
     </gazebo>
+    <gazebo reference="camera_mount">
+      <material>Gazebo/DarkGrey</material>
+    </gazebo>
+    <gazebo reference="camera_interface">
+      <material>Gazebo/DarkGrey</material>
+    </gazebo>
     <!-- Controllers-->
     <!-- <gazebo>
@@ -131,19 +137,3 @@
       </sensor>
   </gazebo>
-  <!-- Realsense Camera-->
-  <!-- <gazebo>
-    <plugin name="realsense_camera" filename="librealsense_gazebo_plugin.so"/>
-      <camera_name>depth_camera</camera_name>
-      <depth_topic>/camera/depth/image_raw</depth_topic>
-      <color_topic>/camera/color/image_raw</color_topic>
-      <infrared1_topic>/camera/infra1/image_raw</infrared1_topic>
-      <infrared2_topic>/camera/infra2/image_raw</infrared2_topic>
-      <depth_camera_info_topic>/camera/depth/camera_info</depth_camera_info_topic>
-      <color_camera_info_topic>/camera/color/camera_info</color_camera_info_topic>
-      <infrared1_camera_info_topic>/camera/infra1/camera_info</infrared1_camera_info_topic>
-      <infrared2_camera_info_topic>/camera/infra2/camera_info</infrared2_camera_info_topic>
-      <pointcloud_topic>/camera/depth/points</pointcloud_topic>
-      <pointcloud_cutoff>0.5</pointcloud_cutoff>
-      <range_max>4.0</range_max>
-  </gazebo> -->
 </robot>

File: mab_description/xacro/silver_badger.urdf.xacro (robot description, xacro)
@@ -18,5 +18,6 @@
   <!-- Initialize camera-->
   <xacro:include filename="$(find mab_description)/xacro/camera.xacro"/>
-  <xacro:realsense2_camera parent="base_link" name="d435_camera"/>
+  <!-- Include camera mount files-->
+  <xacro:include filename="$(find mab_description)/xacro/camera_mount.xacro"/>
   <!-- BODY -->
   <link name="base_link"/>
@@ -35,5 +36,5 @@
       <origin rpy="0 0 0" xyz="0 0 0"/>
       <geometry>
-        <mesh filename="package://meshes/hb40/body.stl" scale="0.001 0.001 0.001"/>
+        <mesh filename="file://$(find mab_description)/meshes/hb40/body.stl" scale="0.001 0.001 0.001"/>
       </geometry>
       <material name="silver"/>
@@ -61,5 +62,5 @@
       <origin rpy="0 0 0" xyz="0 0 0"/>
       <geometry>
-        <mesh filename="package://meshes/hb40/rear.stl" scale="0.001 0.001 0.001"/>
+        <mesh filename="file://$(find mab_description)/meshes/hb40/rear.stl" scale="0.001 0.001 0.001"/>
       </geometry>
       <material name="silver"/>
@@ -77,21 +78,19 @@
     <child link="body"/>
   </joint>
+  <!-- <link name="map"/>
+  <joint name="map_root" type="floating">
+    <parent link="base_link"/>
+    <child link="map"/>
+  </joint> -->
+  <!-- <link name="odom"/>
+  <joint name="odom_root" type="fixed">
+    <parent link="body"/>
+    <child link="odom"/>
+  </joint> -->
+  <!-- Setup IMU-->
   <xacro:imu parent_link="body"/>
-  <!-- <sensor_d435 parent="base_link"/> -->
-  <!-- <link name="realsense_link">
-    <visual>
-      <geometry>
-        <box size="0.1 0.1 0.1"/>
-      </geometry>
-      <material>
-        <color rgba="0 1 0 1"/>
-      </material>
-    </visual>
-  </link>
-  <joint name="realsense_joint" type="fixed">
-    <parent link="base_link"/>
-    <child link="realsense_link"/>
-    <origin xyz="0 0 1.0" rpy="0 0 0"/>
-  </joint> -->
+  <!-- Setup camera mount-->
+  <xacro:realsense2_camera_mount parent="body"/>
+  <xacro:realsense2_camera parent="body" name="d435_camera"/>
   <!-- LEG LINKS 0-4 -->
   <link name="fr_l0">
@@ -109,5 +108,5 @@
       <origin rpy="0 0 0" xyz="0 0 0"/>
       <geometry>
-        <mesh filename="package://meshes/hb40/l0r.stl" scale="0.001 0.001 0.001"/>
+        <mesh filename="file://$(find mab_description)/meshes/hb40/l0r.stl" scale="0.001 0.001 0.001"/>
       </geometry>
       <material name="silver"/>
@@ -128,5 +127,5 @@
       <origin rpy="0 0 0" xyz="0 0 0"/>
       <geometry>
-        <mesh filename="package://meshes/hb40/l1r.stl" scale="0.001 0.001 0.001"/>
+        <mesh filename="file://$(find mab_description)/meshes/hb40/l1r.stl" scale="0.001 0.001 0.001"/>
       </geometry>
       <material name="orange"/>
@@ -153,7 +152,7 @@
       <origin rpy="0 0 0" xyz="0 0 0"/>
       <geometry>
-        <mesh filename="package://meshes/hb40/l2r.stl" scale="0.001 0.001 0.001"/>
-      </geometry>
-      <material name="red"/>
+        <mesh filename="file://$(find mab_description)/meshes/hb40/l2r.stl" scale="0.001 0.001 0.001"/>
+      </geometry>
+      <material name="silver"/>
     </visual>
     <collision>
@@ -206,5 +205,5 @@
       <origin rpy="0 0 0" xyz="0 0 0"/>
       <geometry>
-        <mesh filename="package://meshes/hb40/l0l.stl" scale="0.001 0.001 0.001"/>
+        <mesh filename="file://$(find mab_description)/meshes/hb40/l0l.stl" scale="0.001 0.001 0.001"/>
       </geometry>
       <material name="silver"/>
@@ -225,5 +224,5 @@
       <origin rpy="0 0 0" xyz="0 0 0"/>
       <geometry>
-        <mesh filename="package://meshes/hb40/l1lf.stl" scale="0.001 0.001 0.001"/>
+        <mesh filename="file://$(find mab_description)/meshes/hb40/l1lf.stl" scale="0.001 0.001 0.001"/>
       </geometry>
       <material name="orange"/>
@@ -250,5 +249,5 @@
       <origin rpy="0 0 0" xyz="0 0 0"/>
       <geometry>
-        <mesh filename="package://meshes/hb40/l2l.stl" scale="0.001 0.001 0.001"/>
+        <mesh filename="file://$(find mab_description)/meshes/hb40/l2l.stl" scale="0.001 0.001 0.001"/>
       </geometry>
       <material name="silver"/>
@@ -303,5 +302,5 @@
       <origin rpy="0 0 0" xyz="0 0 0"/>
       <geometry>
-        <mesh filename="package://meshes/hb40/l0l.stl" scale="0.001 0.001 0.001"/>
+        <mesh filename="file://$(find mab_description)/meshes/hb40/l0l.stl" scale="0.001 0.001 0.001"/>
       </geometry>
       <material name="silver"/>
@@ -322,5 +321,5 @@
       <origin rpy="0 0 0" xyz="0 0 0"/>
       <geometry>
-        <mesh filename="package://meshes/hb40/l1lf.stl" scale="0.001 0.001 0.001"/>
+        <mesh filename="file://$(find mab_description)/meshes/hb40/l1lf.stl" scale="0.001 0.001 0.001"/>
       </geometry>
       <material name="orange"/>
@@ -347,5 +346,5 @@
       <origin rpy="0 0 0" xyz="0 0 0"/>
       <geometry>
-        <mesh filename="package://meshes/hb40/l2l.stl" scale="0.001 0.001 0.001"/>
+        <mesh filename="file://$(find mab_description)/meshes/hb40/l2l.stl" scale="0.001 0.001 0.001"/>
       </geometry>
       <material name="silver"/>
@@ -400,5 +399,5 @@
       <origin rpy="0 0 0" xyz="0 0 0"/>
       <geometry>
-        <mesh filename="package://meshes/hb40/l0r.stl" scale="0.001 0.001 0.001"/>
+        <mesh filename="file://$(find mab_description)/meshes/hb40/l0r.stl" scale="0.001 0.001 0.001"/>
       </geometry>
       <material name="silver"/>
@@ -419,5 +418,5 @@
       <origin rpy="0 0 0" xyz="0 0 0"/>
       <geometry>
-        <mesh filename="package://meshes/hb40/l1r.stl" scale="0.001 0.001 0.001"/>
+        <mesh filename="file://$(find mab_description)/meshes/hb40/l1r.stl" scale="0.001 0.001 0.001"/>
       </geometry>
       <material name="orange"/>
@@ -444,5 +443,5 @@
       <origin rpy="0 0 0" xyz="0 0 0"/>
       <geometry>
-        <mesh filename="package://meshes/hb40/l2r.stl" scale="0.001 0.001 0.001"/>
+        <mesh filename="file://$(find mab_description)/meshes/hb40/l2r.stl" scale="0.001 0.001 0.001"/>
       </geometry>
       <material name="silver"/>
