Commit message: slam works with rtabmap - system is laggy on my workstation though

File: mab_description/urdf/silver_badger.urdf (robot description, URDF)
Before this commit: robot silver_badger, 33 links, 32 joints
Links:
- removed link d435_camera__bottom_screw_frame
- removed link d435_camera__color_frame
- removed link d435_camera__color_optical_frame
- removed link d435_camera__depth_frame
- removed link d435_camera__depth_optical_frame
- removed link d435_camera__infra1_frame
- removed link d435_camera__infra1_optical_frame
- removed link d435_camera__infra2_frame
- removed link d435_camera__infra2_optical_frame
- removed link d435_camera__link
- removed link d435_camera__usb_plug_link
- added link camera_image_link, mass 0
- added link d435_camera_bottom_screw_frame
- added link d435_camera_color_frame
- added link d435_camera_color_optical_frame
- added link d435_camera_depth_frame
- added link d435_camera_depth_optical_frame
- added link d435_camera_infra1_frame
- added link d435_camera_infra1_optical_frame
- added link d435_camera_infra2_frame
- added link d435_camera_infra2_optical_frame
- added link d435_camera_link, mass 0.072; collision box size=0.02505 0.09 0.025; visual mesh filename=file:///home/aditya/ros2_ws/install/realsense2_description/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
- added link laser_frame
- added link odom
- link body: geometry collision box size=0.22 0.2 0.1; visual mesh filename=file:///home/aditya/ros2_ws/install/mab_description/share/m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 scale=0.001 0.001 0.001
- link camera_interface: geometry visual mesh filename=file:///home/aditya/ros2_ws/install/mab_description/share/m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 scale=0.001 0.001 0.001
- link camera_mount: geometry visual mesh filename=file:///home/aditya/ros2_ws/install/mab_description/share/m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
- link fl_l0: geometry visual mesh filename=file:///home/aditya/ros2_ws/install/mab_description/share/m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 scale=0.001 0.001 0.001
- link fl_l1: geometry collision cylinder length=0.08 radius=0.05; visual mesh filename=file:///home/aditya/ros2_ws/install/mab_description/share/m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 scale=0.001 0.001 0.001
- link fl_l2: geometry collision cylinder length=0.0625 radius=0.01; collision cylinder length=0.2 radius=0.015
- link fr_l0: geometry visual mesh filename=file:///home/aditya/ros2_ws/install/mab_description/share/m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 scale=0.001 0.001 0.001
- link fr_l1: geometry collision cylinder length=0.08 radius=0.05; visual mesh filename=file:///home/aditya/ros2_ws/install/mab_description/share/m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 scale=0.001 0.001 0.001
- link fr_l2: geometry collision cylinder length=0.0625 radius=0.01; collision cylinder length=0.2 radius=0.015
- link rear: geometry collision box size=0.2 0.05 0.1; visual mesh filename=file:///home/aditya/ros2_ws/install/mab_description/share/m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 scale=0.001 0.001 0.001
- link rl_l0: geometry visual mesh filename=file:///home/aditya/ros2_ws/install/mab_description/share/m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 scale=0.001 0.001 0.001
- link rl_l1: geometry collision cylinder length=0.08 radius=0.05; visual mesh filename=file:///home/aditya/ros2_ws/install/mab_description/share/m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 scale=0.001 0.001 0.001
- link rl_l2: geometry collision cylinder length=0.0625 radius=0.01; collision cylinder length=0.2 radius=0.015
- link rr_l0: geometry visual mesh filename=file:///home/aditya/ros2_ws/install/mab_description/share/m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 scale=0.001 0.001 0.001
- link rr_l1: geometry collision cylinder length=0.08 radius=0.05; visual mesh filename=file:///home/aditya/ros2_ws/install/mab_description/share/m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 scale=0.001 0.001 0.001
- link rr_l2: geometry collision cylinder length=0.0625 radius=0.01; collision cylinder length=0.2 radius=0.015
Joints:
- removed joint d435_camera__color_joint
- removed joint d435_camera__color_optical_joint
- removed joint d435_camera__depth_joint
- removed joint d435_camera__depth_optical_joint
- removed joint d435_camera__infra1_joint
- removed joint d435_camera__infra1_optical_joint
- removed joint d435_camera__infra2_joint
- removed joint d435_camera__infra2_optical_joint
- removed joint d435_camera__joint
- removed joint d435_camera__link_joint
- removed joint d435_camera__usb_plug_joint
- removed joint root
- added joint camera_image_joint: type fixed, parent body, child camera_image_link, origin xyz=0.290755 5.3e-05 0.068583 rpy=-1.5707963267948966 0 0
- added joint d435_camera_color_joint: type fixed, parent d435_camera_link, child d435_camera_color_frame, origin xyz=0 0.015 0 rpy=0 0 0
- added joint d435_camera_color_optical_joint: type fixed, parent d435_camera_color_frame, child d435_camera_color_optical_frame, origin xyz=0 0 0 rpy=-1.5707963267948966 0 -1.5707963267948966
- added joint d435_camera_depth_joint: type fixed, parent d435_camera_link, child d435_camera_depth_frame, origin xyz=0 0 0 rpy=0 0 0
- added joint d435_camera_depth_optical_joint: type fixed, parent d435_camera_depth_frame, child d435_camera_depth_optical_frame, origin xyz=0 0 0 rpy=-1.5707963267948966 0 -1.5707963267948966
- added joint d435_camera_infra1_joint: type fixed, parent d435_camera_link, child d435_camera_infra1_frame, origin xyz=0 0.0 0 rpy=0 0 0
- added joint d435_camera_infra1_optical_joint: type fixed, parent d435_camera_infra1_frame, child d435_camera_infra1_optical_frame, origin xyz=0 0 0 rpy=-1.5707963267948966 0 -1.5707963267948966
- added joint d435_camera_infra2_joint: type fixed, parent d435_camera_link, child d435_camera_infra2_frame, origin xyz=0 -0.05 0 rpy=0 0 0
- added joint d435_camera_infra2_optical_joint: type fixed, parent d435_camera_infra2_frame, child d435_camera_infra2_optical_frame, origin xyz=0 0 0 rpy=-1.5707963267948966 0 -1.5707963267948966
- added joint d435_camera_joint: type fixed, parent body, child d435_camera_bottom_screw_frame, origin xyz=0.275855 -0.012447000000000001 0.068583 rpy=-1.5707963267948966 0 0
- added joint d435_camera_link_joint: type fixed, parent d435_camera_bottom_screw_frame, child d435_camera_link, origin xyz=0.010600000000000002 0.0175 0.0125 rpy=0 0 0
- added joint laser_joint: type fixed, parent camera_image_link, child laser_frame, origin xyz=0 0 0 rpy=1.5707963267948966 0 0
- added joint root1: type fixed, parent odom, child base_link
- added joint root2: type fixed, parent base_link, child body

File: mab_description/xacro/camera.xacro (robot description, xacro)
@@ -25,5 +25,5 @@
         <!-- Initialize camera-->
         <xacro:include filename="$(find realsense2_description)/urdf/_d435.urdf.xacro"/>
-        <xacro:sensor_d435 parent="${parent}" name="${name}" use_nominal_extrinsics="false">
+        <xacro:sensor_d435 parent="${parent}" name="${name}" use_nominal_extrinsics="true">
             <origin xyz="${0.290755-d435_mesh_x_offset-d435_zero_depth_to_glass - d435_glass_to_front} ${0.000053-d435_cam_depth_pz} ${0.068583}" rpy="${-M_PI/2} 0 0"/>
         </xacro:sensor_d435>
@@ -44,4 +44,10 @@
             <origin rpy="${d435_cam_roll} 0 0" xyz="${d435_cam_x} ${d435_cam_y} ${d435_cam_z}" />
         </joint>
+        <link name="laser_frame"/>
+        <joint name="laser_joint" type="fixed">
+            <parent link="camera_image_link"/>
+            <child link="laser_frame"/>
+            <origin rpy="${-d435_cam_roll} 0 0" xyz="0 0 0"/>
+        </joint>
         <!-- Some parameters-->
         <xacro:property name="camera_name" value="${name}" />
@@ -55,4 +61,5 @@
         <!-- Load parameters to model's main link-->
         <xacro:property name="deg_to_rad" value="0.01745329251994329577" />
+        <!-- <gazebo reference="camera_image_link"> -->
         <gazebo reference="camera_image_link">
             <self_collide>0</self_collide>
@@ -139,6 +146,6 @@
                     <horizontal_fov>${85.2*deg_to_rad}</horizontal_fov>
                     <image>
-                        <width>1280</width>
-                        <height>720</height>
+                        <width>640</width>
+                        <height>480</height>
                     </image>
                     <clip>

File: mab_description/xacro/silver_badger.urdf.xacro (robot description, xacro)
@@ -11,9 +11,9 @@
   <xacro:include filename="$(find mab_description)/xacro/materials.xacro" />
   <!-- Import control tags-->
-  <xacro:include filename="$(find mab_description)/xacro/control.xacro" />
+  <!-- <xacro:include filename="$(find mab_description)/xacro/control.xacro" /> -->
   <!-- Include limits-->
   <xacro:include filename="$(find mab_description)/xacro/limits.xacro" />
   <!-- Initialize controls-->
-  <xacro:silver_badger_ros2_control/>
+  <!-- <xacro:silver_badger_ros2_control/> -->
   <!-- Initialize camera-->
   <xacro:include filename="$(find mab_description)/xacro/camera.xacro"/>
@@ -85,5 +85,5 @@
   <!-- <link name="odom"/>
   <joint name="odom_root" type="fixed">
-    <parent link="body"/>
+    <parent link="base_link"/>
     <child link="odom"/>
   </joint> -->

Commit message: added bringup package and tuned slam

File: mab_description/urdf/silver_badger.urdf (robot description, URDF)
Before this commit: robot silver_badger, 35 links, 34 joints
Links:
- removed link d435_camera_bottom_screw_frame
- removed link d435_camera_color_frame
- removed link d435_camera_color_optical_frame
- removed link d435_camera_depth_frame
- removed link d435_camera_depth_optical_frame
- removed link d435_camera_infra1_frame
- removed link d435_camera_infra1_optical_frame
- removed link d435_camera_infra2_frame
- removed link d435_camera_infra2_optical_frame
- removed link d435_camera_link
- removed link odom
- added link d435i_camera_accel_frame
- added link d435i_camera_accel_optical_frame
- added link d435i_camera_bottom_screw_frame
- added link d435i_camera_color_frame
- added link d435i_camera_color_optical_frame
- added link d435i_camera_depth_frame
- added link d435i_camera_depth_optical_frame
- added link d435i_camera_gyro_frame
- added link d435i_camera_gyro_optical_frame
- added link d435i_camera_infra1_frame
- added link d435i_camera_infra1_optical_frame
- added link d435i_camera_infra2_frame
- added link d435i_camera_infra2_optical_frame
- added link d435i_camera_link, mass 0.072; collision box size=0.02505 0.09 0.025; visual mesh filename=file:///home/aditya/ros2_ws/install/realsense2_description/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
Joints:
- removed joint d435_camera_color_joint
- removed joint d435_camera_color_optical_joint
- removed joint d435_camera_depth_joint
- removed joint d435_camera_depth_optical_joint
- removed joint d435_camera_infra1_joint
- removed joint d435_camera_infra1_optical_joint
- removed joint d435_camera_infra2_joint
- removed joint d435_camera_infra2_optical_joint
- removed joint d435_camera_joint
- removed joint d435_camera_link_joint
- removed joint root1
- removed joint root2
- added joint d435i_camera_accel_joint: type fixed, parent d435i_camera_link, child d435i_camera_accel_frame, origin xyz=-0.01174 -0.00552 0.0051 rpy=0 0 0
- added joint d435i_camera_accel_optical_joint: type fixed, parent d435i_camera_accel_frame, child d435i_camera_accel_optical_frame, origin xyz=0 0 0 rpy=-1.5707963267948966 0 -1.5707963267948966
- added joint d435i_camera_color_joint: type fixed, parent d435i_camera_link, child d435i_camera_color_frame, origin xyz=0 0.015 0 rpy=0 0 0
- added joint d435i_camera_color_optical_joint: type fixed, parent d435i_camera_color_frame, child d435i_camera_color_optical_frame, origin xyz=0 0 0 rpy=-1.5707963267948966 0 -1.5707963267948966
- added joint d435i_camera_depth_joint: type fixed, parent d435i_camera_link, child d435i_camera_depth_frame, origin xyz=0 0 0 rpy=0 0 0
- added joint d435i_camera_depth_optical_joint: type fixed, parent d435i_camera_depth_frame, child d435i_camera_depth_optical_frame, origin xyz=0 0 0 rpy=-1.5707963267948966 0 -1.5707963267948966
- added joint d435i_camera_gyro_joint: type fixed, parent d435i_camera_link, child d435i_camera_gyro_frame, origin xyz=-0.01174 -0.00552 0.0051 rpy=0 0 0
- added joint d435i_camera_gyro_optical_joint: type fixed, parent d435i_camera_gyro_frame, child d435i_camera_gyro_optical_frame, origin xyz=0 0 0 rpy=-1.5707963267948966 0 -1.5707963267948966
- added joint d435i_camera_infra1_joint: type fixed, parent d435i_camera_link, child d435i_camera_infra1_frame, origin xyz=0 0.0 0 rpy=0 0 0
- added joint d435i_camera_infra1_optical_joint: type fixed, parent d435i_camera_infra1_frame, child d435i_camera_infra1_optical_frame, origin xyz=0 0 0 rpy=-1.5707963267948966 0 -1.5707963267948966
- added joint d435i_camera_infra2_joint: type fixed, parent d435i_camera_link, child d435i_camera_infra2_frame, origin xyz=0 -0.05 0 rpy=0 0 0
- added joint d435i_camera_infra2_optical_joint: type fixed, parent d435i_camera_infra2_frame, child d435i_camera_infra2_optical_frame, origin xyz=0 0 0 rpy=-1.5707963267948966 0 -1.5707963267948966
- added joint d435i_camera_joint: type fixed, parent body, child d435i_camera_bottom_screw_frame, origin xyz=0.275855 -0.012447000000000001 0.068583 rpy=-1.5707963267948966 0 0
- added joint d435i_camera_link_joint: type fixed, parent d435i_camera_bottom_screw_frame, child d435i_camera_link, origin xyz=0.010600000000000002 0.0175 0.0125 rpy=0 0 0
- added joint root: type fixed, parent base_link, child body

File: mab_description/xacro/camera.xacro (robot description, xacro)
@@ -23,9 +23,11 @@
         <xacro:property name="d435_cam_z" value="0.068583"/>
         <xacro:property name="d435_cam_roll" value="${-M_PI/2}"/>
+        <!-- <xacro:property name="d435_cam_roll" value="0"/> -->
         <!-- Initialize camera-->
-        <xacro:include filename="$(find realsense2_description)/urdf/_d435.urdf.xacro"/>
-        <xacro:sensor_d435 parent="${parent}" name="${name}" use_nominal_extrinsics="true">
-            <origin xyz="${0.290755-d435_mesh_x_offset-d435_zero_depth_to_glass - d435_glass_to_front} ${0.000053-d435_cam_depth_pz} ${0.068583}" rpy="${-M_PI/2} 0 0"/>
-        </xacro:sensor_d435>
+        <xacro:include filename="$(find realsense2_description)/urdf/_d435i.urdf.xacro"/>
+        <xacro:sensor_d435i parent="${parent}" name="${name}" use_nominal_extrinsics="true">
+            <!-- <origin xyz="${0.290755-d435_mesh_x_offset-d435_zero_depth_to_glass - d435_glass_to_front} ${0.000053-d435_cam_depth_pz} ${0.068583}" rpy="${0} 0 0"/> -->
+            <origin xyz="${0.290755-d435_mesh_x_offset-d435_zero_depth_to_glass - d435_glass_to_front} ${0.000053-d435_cam_depth_pz} ${0.068583}" rpy="${d435_cam_roll} 0 0"/>
+        </xacro:sensor_d435i>
         <!-- Link for camera image and gazebe plugin-->
         <link name="camera_image_link">
@@ -80,4 +82,6 @@
                     <horizontal_fov>${69.4*deg_to_rad}</horizontal_fov>
                     <image>
+                        <!-- <width>1280</width>
+                        <height>720</height> -->
                         <width>640</width>
                         <height>480</height>
@@ -95,5 +99,5 @@
                 </camera>
                 <always_on>1</always_on>
-                <update_rate>30</update_rate>
+                <update_rate>90</update_rate>
                 <visualize>1</visualize>
             </sensor>
@@ -146,4 +150,6 @@
                     <horizontal_fov>${85.2*deg_to_rad}</horizontal_fov>
                     <image>
+                        <!-- <width>1280</width>
+                        <height>720</height> -->
                         <width>640</width>
                         <height>480</height>
@@ -167,6 +173,6 @@
             <plugin name="${topics_ns}" filename="librealsense_gazebo_plugin.so">
                 <prefix>${camera_name}</prefix>
-                <depthUpdateRate>30.0</depthUpdateRate>
-                <colorUpdateRate>30.0</colorUpdateRate>
+                <depthUpdateRate>90.0</depthUpdateRate>
+                <colorUpdateRate>90.0</colorUpdateRate>
                 <infraredUpdateRate>0.0</infraredUpdateRate>
                 <depthTopicName>${topics_ns}/depth/image_raw</depthTopicName>

File: mab_description/xacro/silver_badger.gazebo.xacro (robot description, xacro)
@@ -120,9 +120,11 @@
     </gazebo>
     <!-- Sensors-->
+    <xacro:property name="M_PI" value="3.1415926535897931" />
     <gazebo reference="imu_link">
+    <!-- <gazebo reference="d435i_camera_accel_frame"> -->
       <gravity>true</gravity>
       <sensor name='imu_sensor' type='imu'>
           <always_on>1</always_on>
-          <update_rate>20</update_rate>
+          <update_rate>100</update_rate>
           <visualize>1</visualize>
           <topic>imu</topic>
@@ -130,5 +132,5 @@
               <topicName>imu</topicName>
               <bodyName>imu_sensor_link</bodyName>
-              <updateRateHZ>20.0</updateRateHZ>
+              <updateRateHZ>100.0</updateRateHZ>
               <xyzOffset>0 0 0</xyzOffset>
               <rpyOffset>0 0 0</rpyOffset>
@@ -136,4 +138,21 @@
           <pose>0 0 0 0 0 0</pose>
       </sensor>
-  </gazebo>
+    </gazebo>
+    <!-- <gazebo reference="d435i_camera_accel_frame">
+      <gravity>true</gravity>
+      <sensor name='cam_imu_sensor' type='imu'>
+          <always_on>1</always_on>
+          <update_rate>100</update_rate>
+          <visualize>1</visualize>
+          <topic>cam_imu</topic>
+          <plugin name='cam_imu' filename='libgazebo_ros_imu_sensor.so'>
+              <topicName>cam_imu</topicName>
+              <bodyName>cam_imu_sensor_link</bodyName>
+              <updateRateHZ>100.0</updateRateHZ>
+              <xyzOffset>0 0 0</xyzOffset>
+              <rpyOffset>0 0 0</rpyOffset>
+          </plugin>
+          <pose>0 0 0 0 0 0</pose>
+      </sensor>
+    </gazebo> -->
 </robot>

File: mab_description/xacro/silver_badger.urdf.xacro (robot description, xacro)
@@ -88,9 +88,9 @@
     <child link="odom"/>
   </joint> -->
+  <!-- Setup camera mount-->
+  <xacro:realsense2_camera_mount parent="body"/>
+  <xacro:realsense2_camera parent="body" name="d435i_camera"/>
   <!-- Setup IMU-->
   <xacro:imu parent_link="body"/>
-  <!-- Setup camera mount-->
-  <xacro:realsense2_camera_mount parent="body"/>
-  <xacro:realsense2_camera parent="body" name="d435_camera"/>
   <!-- LEG LINKS 0-4 -->
   <link name="fr_l0">
