Commit message: final commit from IAS

File: mab_description/urdf/honey_badger.urdf (robot description, URDF)
Before this commit: robot honey_badger, 37 links, 36 joints
Links:
- link laser_frame: mass 0 -> None
Joints:
- removed joint laser_frame_joint
- added joint laser_joint: type fixed, parent camera_image_link, child laser_frame, origin xyz=0 0 0 rpy=1.5707963267948966 0 0
- joint fl_j0: type continuous -> revolute
- joint fl_j1: type continuous -> revolute
- joint fl_j2: type continuous -> revolute
- joint fr_j0: type continuous -> revolute
- joint fr_j1: type continuous -> revolute
- joint fr_j2: type continuous -> revolute
- joint rl_j0: type continuous -> revolute
- joint rl_j1: type continuous -> revolute
- joint rl_j2: type continuous -> revolute
- joint rr_j0: type continuous -> revolute
- joint rr_j1: type continuous -> revolute
- joint rr_j2: type continuous -> revolute

File: mab_description/urdf/silver_badger.urdf (robot description, URDF)
Before this commit: robot silver_badger, 38 links, 37 joints
Joints:
- joint fl_j0: type continuous -> revolute
- joint fl_j1: type continuous -> revolute
- joint fl_j2: type continuous -> revolute
- joint fr_j0: type continuous -> revolute
- joint fr_j1: type continuous -> revolute
- joint fr_j2: type continuous -> revolute
- joint rl_j0: type continuous -> revolute
- joint rl_j1: type continuous -> revolute
- joint rl_j2: type continuous -> revolute
- joint rr_j0: type continuous -> revolute
- joint rr_j1: type continuous -> revolute
- joint rr_j2: type continuous -> revolute
- joint sp_j0: type continuous -> revolute

File: mab_description/xacro/gazebo.xacro (robot description, xacro)
@@ -138,4 +138,5 @@
               <xyzOffset>0 0 0</xyzOffset>
               <rpyOffset>0 0 0</rpyOffset>
+              <gaussianNoise>0.017</gaussianNoise>
           </plugin>
           <pose>0 0 0 0 0 0</pose>
@@ -159,4 +160,83 @@
       </sensor>
     </gazebo> -->
+    <!-- Foot Contact Sensors-->
+    <gazebo reference="fr_foot">
+      <sensor name="fr_foot_bumper" type="contact">
+          <selfCollide>true</selfCollide>
+          <alwaysOn>true</alwaysOn>
+          <updateRate>50.0</updateRate>
+          <material>Gazebo/Red</material>
+          <contact>
+              <collision>fr_l2_fixed_joint_lump__fr_foot_collision_2</collision>
+          </contact>
+          <plugin name="gazebo_ros_bumper_controller_fr_foot" filename="libgazebo_ros_bumper.so">
+              <ros>
+                  <remapping>bumper_states:=feet_contact</remapping>
+              </ros>
+          </plugin>
+      </sensor>
+  </gazebo>
+  <gazebo reference="fl_foot">
+      <sensor name="fl_foot_bumper" type="contact">
+          <selfCollide>true</selfCollide>
+          <alwaysOn>true</alwaysOn>
+          <updateRate>50.0</updateRate>
+          <material>Gazebo/Red</material>
+          <contact>
+              <collision>fl_l2_fixed_joint_lump__fl_foot_collision_2</collision>
+          </contact>
+          <plugin name="gazebo_ros_bumper_controller_fl_foot" filename="libgazebo_ros_bumper.so">
+              <ros>
+                  <remapping>bumper_states:=feet_contact</remapping>
+              </ros>
+          </plugin>
+      </sensor>
+  </gazebo>
+  <gazebo reference="rr_foot">
+    <sensor name="rr_foot_bumper" type="contact">
+        <selfCollide>true</selfCollide>
+        <alwaysOn>true</alwaysOn>
+        <updateRate>50.0</updateRate>
+        <material>Gazebo/Red</material>
+        <contact>
+            <collision>rr_l2_fixed_joint_lump__rr_foot_collision_2</collision>
+        </contact>
+        <plugin name="gazebo_ros_bumper_controller_rr_foot" filename="libgazebo_ros_bumper.so">
+            <ros>
+                <remapping>bumper_states:=feet_contact</remapping>
+            </ros>
+        </plugin>
+    </sensor>
+  </gazebo>
+  <gazebo reference="rl_foot">
+    <sensor name="rl_foot_bumper" type="contact">
+        <selfCollide>true</selfCollide>
+        <alwaysOn>true</alwaysOn>
+        <updateRate>50.0</updateRate>
+        <material>Gazebo/Red</material>
+        <contact>
+            <collision>rl_l2_fixed_joint_lump__rl_foot_collision_2</collision>
+        </contact>
+        <plugin name="gazebo_ros_bumper_controller_rl_foot" filename="libgazebo_ros_bumper.so">
+            <ros>
+                <remapping>bumper_states:=feet_contact</remapping>
+            </ros>
+        </plugin>
+    </sensor>
+  </gazebo>
+  <!-- Ground truth odom-->
+  <gazebo>
+    <plugin name="gazebo_ros_p3d" filename="libgazebo_ros_p3d.so">
+      <ros>
+        <remapping>odom:=odom_gt</remapping>
+      </ros>
+      <body_name>base_link</body_name>
+      <frame_name>world</frame_name>
+      <update_rate>100</update_rate>
+      <xyz_offset>0 0 0</xyz_offset>
+      <rpy_offset>0 0 0</rpy_offset>
+      <gaussian_noise>0.0</gaussian_noise>
+    </plugin>
+  </gazebo>
   </xacro:macro>
 </robot>

File: mab_description/xacro/honey_badger.urdf.xacro (robot description, xacro)
@@ -451,5 +451,5 @@
   <!-- LEGS JOINTS 0-4  -->
   <!-- Front Right Leg -->
-  <joint armature="0.01" name="fr_j0" type="continuous">
+  <joint armature="0.01" name="fr_j0" type="revolute">
     <parent link="body"/>
     <child link="fr_l0"/>
@@ -458,5 +458,5 @@
     <limit effort="${fr_j0_max_effort}" lower="${fr_j0_limit_lower}" upper="${fr_j0_limit_upper}" velocity="${fr_j0_max_velocity}"/>
   </joint>
-  <joint name="fr_j1" type="continuous">
+  <joint name="fr_j1" type="revolute">
     <parent link="fr_l0"/>
     <child link="fr_l1"/>
@@ -465,5 +465,5 @@
     <limit effort="${fr_j1_max_effort}" lower="${fr_j1_limit_lower}" upper="${fr_j1_limit_upper}" velocity="${fr_j1_max_velocity}"/>
   </joint>
-  <joint name="fr_j2" type="continuous">
+  <joint name="fr_j2" type="revolute">
     <parent link="fr_l1"/>
     <child link="fr_l2"/>
@@ -479,5 +479,5 @@
   </joint>
   <!-- Front Left Leg -->
-  <joint armature="0.01" name="fl_j0" type="continuous">
+  <joint armature="0.01" name="fl_j0" type="revolute">
     <parent link="body"/>
     <child link="fl_l0"/>
@@ -486,5 +486,5 @@
     <limit effort="${fl_j0_max_effort}" lower="${fl_j0_limit_lower}" upper="${fl_j0_limit_upper}" velocity="${fl_j0_max_velocity}"/>
   </joint>
-  <joint name="fl_j1" type="continuous">
+  <joint name="fl_j1" type="revolute">
     <parent link="fl_l0"/>
     <child link="fl_l1"/>
@@ -493,5 +493,5 @@
     <limit effort="${fl_j1_max_effort}" lower="${fl_j1_limit_lower}" upper="${fl_j1_limit_upper}" velocity="${fl_j1_max_velocity}"/>
   </joint>
-  <joint name="fl_j2" type="continuous">
+  <joint name="fl_j2" type="revolute">
     <parent link="fl_l1"/>
     <child link="fl_l2"/>
@@ -507,5 +507,5 @@
   </joint>
   <!-- Rear Left Leg -->
-  <joint armature="0.01" name="rl_j0" type="continuous">
+  <joint armature="0.01" name="rl_j0" type="revolute">
     <parent link="body"/>
     <child link="rl_l0"/>
@@ -514,5 +514,5 @@
     <limit effort="${rl_j0_max_effort}" lower="${rl_j0_limit_lower}" upper="${rl_j0_limit_upper}" velocity="${rl_j0_max_velocity}"/>
   </joint>
-  <joint name="rl_j1" type="continuous">
+  <joint name="rl_j1" type="revolute">
     <parent link="rl_l0"/>
     <child link="rl_l1"/>
@@ -521,5 +521,5 @@
     <limit effort="${rl_j1_max_effort}" lower="${rl_j1_limit_lower}" upper="${rl_j1_limit_upper}" velocity="${rl_j1_max_velocity}"/>
   </joint>
-  <joint name="rl_j2" type="continuous">
+  <joint name="rl_j2" type="revolute">
     <parent link="rl_l1"/>
     <child link="rl_l2"/>
@@ -535,5 +535,5 @@
   </joint>
   <!-- Rear Right Leg -->
-  <joint armature="0.01" name="rr_j0" type="continuous">
+  <joint armature="0.01" name="rr_j0" type="revolute">
     <parent link="body"/>
     <child link="rr_l0"/>
@@ -542,5 +542,5 @@
     <limit effort="${rr_j0_max_effort}" lower="${rr_j0_limit_lower}" upper="${rr_j0_limit_upper}" velocity="${rr_j0_max_velocity}"/>
   </joint>
-  <joint name="rr_j1" type="continuous">
+  <joint name="rr_j1" type="revolute">
     <parent link="rr_l0"/>
     <child link="rr_l1"/>
@@ -549,5 +549,5 @@
     <limit effort="${rr_j1_max_effort}" lower="${rr_j1_limit_lower}" upper="${rr_j1_limit_upper}" velocity="${rr_j1_max_velocity}"/>
   </joint>
-  <joint name="rr_j2" type="continuous">
+  <joint name="rr_j2" type="revolute">
     <parent link="rr_l1"/>
     <child link="rr_l2"/>

File: mab_description/xacro/silver_badger.urdf.xacro (robot description, xacro)
@@ -475,5 +475,5 @@
   <!-- LEG JOINTS 0-4 -->
   <!-- Front Right Leg -->
-  <joint armature="0.01" name="fr_j0" type="continuous">
+  <joint armature="0.01" name="fr_j0" type="revolute">
     <parent link="body"/>
     <child link="fr_l0"/>
@@ -482,5 +482,5 @@
     <limit effort="${fr_j0_max_effort}" lower="${fr_j0_limit_lower}" upper="${fr_j0_limit_upper}" velocity="${fr_j0_max_velocity}"/>
   </joint>
-  <joint name="fr_j1" type="continuous">
+  <joint name="fr_j1" type="revolute">
     <parent link="fr_l0"/>
     <child link="fr_l1"/>
@@ -489,5 +489,5 @@
     <limit effort="${fr_j1_max_effort}" lower="${fr_j1_limit_lower}" upper="${fr_j1_limit_upper}" velocity="${fr_j1_max_velocity}"/>
   </joint>
-  <joint name="fr_j2" type="continuous">
+  <joint name="fr_j2" type="revolute">
     <parent link="fr_l1"/>
     <child link="fr_l2"/>
@@ -503,5 +503,5 @@
   </joint>
   <!-- Front Left Leg -->
-  <joint armature="0.01" name="fl_j0" type="continuous">
+  <joint armature="0.01" name="fl_j0" type="revolute">
     <parent link="body"/>
     <child link="fl_l0"/>
@@ -510,5 +510,5 @@
     <limit effort="${fl_j0_max_effort}" lower="${fl_j0_limit_lower}" upper="${fl_j0_limit_upper}" velocity="${fl_j0_max_velocity}"/>
   </joint>
-  <joint name="fl_j1" type="continuous">
+  <joint name="fl_j1" type="revolute">
     <parent link="fl_l0"/>
     <child link="fl_l1"/>
@@ -517,5 +517,5 @@
     <limit effort="${fl_j1_max_effort}" lower="${fl_j1_limit_lower}" upper="${fl_j1_limit_upper}" velocity="${fl_j1_max_velocity}"/>
   </joint>
-  <joint name="fl_j2" type="continuous">
+  <joint name="fl_j2" type="revolute">
     <parent link="fl_l1"/>
     <child link="fl_l2"/>
@@ -531,5 +531,5 @@
   </joint>
   <!-- Rear Left Leg -->
-  <joint armature="0.01" name="rl_j0" type="continuous">
+  <joint armature="0.01" name="rl_j0" type="revolute">
     <parent link="rear"/>
     <child link="rl_l0"/>
@@ -538,5 +538,5 @@
     <limit effort="${rl_j0_max_effort}" lower="${rl_j0_limit_lower}" upper="${rl_j0_limit_upper}" velocity="${rl_j0_max_velocity}"/>
   </joint>
-  <joint name="rl_j1" type="continuous">
+  <joint name="rl_j1" type="revolute">
     <parent link="rl_l0"/>
     <child link="rl_l1"/>
@@ -545,5 +545,5 @@
     <limit effort="${rl_j1_max_effort}" lower="${rl_j1_limit_lower}" upper="${rl_j1_limit_upper}" velocity="${rl_j1_max_velocity}"/>
   </joint>
-  <joint name="rl_j2" type="continuous">
+  <joint name="rl_j2" type="revolute">
     <parent link="rl_l1"/>
     <child link="rl_l2"/>
@@ -559,5 +559,5 @@
   </joint>
   <!-- Rear Right Leg -->
-  <joint armature="0.01" name="rr_j0" type="continuous">
+  <joint armature="0.01" name="rr_j0" type="revolute">
     <parent link="rear"/>
     <child link="rr_l0"/>
@@ -566,5 +566,5 @@
     <limit effort="${rr_j0_max_effort}" lower="${rr_j0_limit_lower}" upper="${rr_j0_limit_upper}" velocity="${rr_j0_max_velocity}"/>
   </joint>
-  <joint name="rr_j1" type="continuous">
+  <joint name="rr_j1" type="revolute">
     <parent link="rr_l0"/>
     <child link="rr_l1"/>
@@ -573,5 +573,5 @@
     <limit effort="${rr_j1_max_effort}" lower="${rr_j1_limit_lower}" upper="${rr_j1_limit_upper}" velocity="${rr_j1_max_velocity}"/>
   </joint>
-  <joint name="rr_j2" type="continuous">
+  <joint name="rr_j2" type="revolute">
     <parent link="rr_l1"/>
     <child link="rr_l2"/>
@@ -587,5 +587,5 @@
   </joint>
   <!-- Spine Joint-->
-  <joint name="sp_j0" type="continuous">
+  <joint name="sp_j0" type="revolute">
     <parent link="body"/>
     <child link="rear"/>

Commit message: bug fix for non-zero velocity in static state

File: mab_description/urdf/honey_badger.urdf (robot description, URDF)
Before this commit: robot honey_badger, 37 links, 36 joints
Links:
- link body: geometry collision box size=0.27 0.178 0.1; visual mesh filename=file:///home/junninghuang/ros2_ws/install/mab_description/s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 scale=0.001 0.001 0.001
- link camera_interface: geometry visual mesh filename=file:///home/junninghuang/ros2_ws/install/mab_description/s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 scale=0.001 0.001 0.001
- link camera_mount: geometry visual mesh filename=file:///home/junninghuang/ros2_ws/install/mab_description/s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
- link d435i_camera_link: geometry collision box size=0.02505 0.09 0.025; visual mesh filename=file:///home/junninghuang/ros2_ws/install/realsense2_descri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
- link fl_l0: geometry visual mesh filename=file:///home/junninghuang/ros2_ws/install/mab_description/s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 scale=0.001 0.001 0.001
- link fl_l1: geometry collision cylinder length=0.11 radius=0.05; visual mesh filename=file:///home/junninghuang/ros2_ws/install/mab_description/s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 scale=0.001 0.001 0.001
- link fl_l2: geometry collision cylinder length=0.0625 radius=0.01; collision cylinder length=0.2 radius=0.015
- link fr_l0: geometry visual mesh filename=file:///home/junninghuang/ros2_ws/install/mab_description/s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 scale=0.001 0.001 0.001
- link fr_l1: geometry collision cylinder length=0.11 radius=0.05; visual mesh filename=file:///home/junninghuang/ros2_ws/install/mab_description/s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 scale=0.001 0.001 0.001
- link fr_l2: geometry collision cylinder length=0.0625 radius=0.01; collision cylinder length=0.2 radius=0.015
- link rl_l0: geometry visual mesh filename=file:///home/junninghuang/ros2_ws/install/mab_description/s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 scale=0.001 0.001 0.001
- link rl_l1: geometry collision cylinder length=0.11 radius=0.05; visual mesh filename=file:///home/junninghuang/ros2_ws/install/mab_description/s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 scale=0.001 0.001 0.001
- link rl_l2: geometry collision cylinder length=0.0625 radius=0.01; collision cylinder length=0.2 radius=0.015
- link rr_l0: geometry visual mesh filename=file:///home/junninghuang/ros2_ws/install/mab_description/s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 scale=0.001 0.001 0.001
- link rr_l1: geometry collision cylinder length=0.11 radius=0.05; visual mesh filename=file:///home/junninghuang/ros2_ws/install/mab_description/s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 scale=0.001 0.001 0.001
- link rr_l2: geometry collision cylinder length=0.0625 radius=0.01; collision cylinder length=0.2 radius=0.015

File: mab_description/urdf/silver_badger.urdf (robot description, URDF)
Before this commit: robot silver_badger, 38 links, 37 joints
Links:
- link body: geometry collision box size=0.22 0.2 0.1; visual mesh filename=file:///home/junninghuang/ros2_ws/install/mab_description/s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 scale=0.001 0.001 0.001
- link camera_interface: geometry visual mesh filename=file:///home/junninghuang/ros2_ws/install/mab_description/s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 scale=0.001 0.001 0.001
- link camera_mount: geometry visual mesh filename=file:///home/junninghuang/ros2_ws/install/mab_description/s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
- link d435i_camera_link: geometry collision box size=0.02505 0.09 0.025; visual mesh filename=file:///home/junninghuang/ros2_ws/install/realsense2_descri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
- link fl_l0: geometry visual mesh filename=file:///home/junninghuang/ros2_ws/install/mab_description/s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 scale=0.001 0.001 0.001
- link fl_l1: geometry collision cylinder length=0.08 radius=0.05; visual mesh filename=file:///home/junninghuang/ros2_ws/install/mab_description/s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 scale=0.001 0.001 0.001
- link fl_l2: geometry collision cylinder length=0.0625 radius=0.01; collision cylinder length=0.2 radius=0.015
- link fr_l0: geometry visual mesh filename=file:///home/junninghuang/ros2_ws/install/mab_description/s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 scale=0.001 0.001 0.001
- link fr_l1: geometry collision cylinder length=0.08 radius=0.05; visual mesh filename=file:///home/junninghuang/ros2_ws/install/mab_description/s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 scale=0.001 0.001 0.001
- link fr_l2: geometry collision cylinder length=0.0625 radius=0.01; collision cylinder length=0.2 radius=0.015
- link rear: geometry collision box size=0.2 0.05 0.1; visual mesh filename=file:///home/junninghuang/ros2_ws/install/mab_description/s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 scale=0.001 0.001 0.001
- link rl_l0: geometry visual mesh filename=file:///home/junninghuang/ros2_ws/install/mab_description/s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 scale=0.001 0.001 0.001
- link rl_l1: geometry collision cylinder length=0.08 radius=0.05; visual mesh filename=file:///home/junninghuang/ros2_ws/install/mab_description/s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 scale=0.001 0.001 0.001
- link rl_l2: geometry collision cylinder length=0.0625 radius=0.01; collision cylinder length=0.2 radius=0.015
- link rr_l0: geometry visual mesh filename=file:///home/junninghuang/ros2_ws/install/mab_description/s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 scale=0.001 0.001 0.001
- link rr_l1: geometry collision cylinder length=0.08 radius=0.05; visual mesh filename=file:///home/junninghuang/ros2_ws/install/mab_description/s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 scale=0.001 0.001 0.001
- link rr_l2: geometry collision cylinder length=0.0625 radius=0.01; collision cylinder length=0.2 radius=0.015

File: mab_description/xacro/gazebo.xacro (robot description, xacro)
@@ -32,6 +32,6 @@
       <mu2>0.6</mu2>
       <self_collide>0</self_collide>
-      <kp value="1000000.0"/>
-      <kd value="1.0"/>
+      <kp value="1e15"/>
+      <kd value="1e13"/>
       <material>Gazebo/Black</material>
     </gazebo>
@@ -55,6 +55,6 @@
       <mu2>0.6</mu2>
       <self_collide>0</self_collide>
-      <kp value="1000000.0"/>
-      <kd value="1.0"/>
+      <kp value="1e15"/>
+      <kd value="1e13"/>
       <material>Gazebo/Black</material>
     </gazebo>
@@ -78,6 +78,6 @@
       <mu2>0.6</mu2>
       <self_collide>0</self_collide>
-      <kp value="1000000.0"/>
-      <kd value="1.0"/>
+      <kp value="1e15"/>
+      <kd value="1e13"/>
       <material>Gazebo/Black</material>
     </gazebo>
@@ -101,6 +101,6 @@
       <mu2>0.6</mu2>
       <self_collide>0</self_collide>
-      <kp value="1000000.0"/>
-      <kd value="1.0"/>
+      <kp value="1e15"/>
+      <kd value="1e13"/>
       <material>Gazebo/Black</material>
     </gazebo>
