Commit message: modified inertia origins to COMs (not default ones given by MAB)

File: mab_description/xacro/silver_badger.urdf.xacro (robot description, xacro)
@@ -23,6 +23,5 @@
     </inertial> -->
     <inertial>
-      <!-- <origin xyz="19.23637020e-3 0.65977049e-3 3.38565104e-3"/> -->
-      <origin rpy="0 0 0" xyz="0 0 0"/>
+      <origin xyz="19.23637020e-3 0.65977049e-3 3.38565104e-3"/>
       <mass value="5.42300000"/>
       <inertia ixx="21646.56458935e-6" ixy="-46.55756531e-6" ixz="18.07857599e-6" iyy="40703.39489390e-6" iyz="-71.07150002e-6" izz="54721.98086004e-6"/>
@@ -50,6 +49,5 @@
     </inertial> -->
     <inertial>
-      <!-- <origin xyz="-38.28391582e-3 65.76740154e-3 0.15093929e-3"/> -->
-      <origin rpy="0 0 0" xyz="-0.038 0.075 0"/>
+      <origin xyz="-38.28391582e-3 65.76740154e-3 0.15093929e-3"/>
       <mass value="1.33700000"/>
       <inertia ixx="1982.84311251e-6" ixy="-36.51038588e-6" ixz="-4.15042187e-6" iyy="4644.92962873e-6" iyz="0.10412770e-6" izz="5097.13064643e-6"/>
@@ -89,6 +87,5 @@
     </inertial> -->
     <inertial>
-      <!-- <origin xyz="50.33286050e-3 11.96674461e-3 0.45712186e-3"/> -->
-      <origin rpy="0 0 0" xyz="0.0557 -0.016 0"/>
+      <origin xyz="50.33286050e-3 11.96674461e-3 0.45712186e-3"/>
       <mass value="0.64500000"/>
       <inertia ixx="498.32637726e-6" ixy="-43.44106123e-6" ixz="-0.22311702e-6" iyy="842.25430777e-6" iyz="-0.01118942e-6" izz="586.98453014e-6"/>
@@ -109,6 +106,5 @@
     </inertial> -->
     <inertial>
-      <!-- <origin xyz="41.97647538e-3 -50.28912232e-3 5.24458524e-3"/> -->
-      <origin rpy="0 0 0" xyz="0.031 -0.016 0"/>
+      <origin xyz="41.97647538e-3 -50.28912232e-3 5.24458524e-3"/>
       <mass value="0.82700000"/>
       <inertia ixx="4027.34053636e-6" ixy="339.60345125e-6" ixz="-19.19423339e-6" iyy="719.63841788e-6" iyz="70.69913102e-6" izz="3870.59006761e-6"/>
@@ -135,6 +131,5 @@
     </inertial> -->
     <inertial>
-      <!-- <origin xyz="1.42261228e-3 -96.66711845e-3 1.53962525e-3"/> -->
-      <origin rpy="0 0 0" xyz="0.001 -0.104 -0.003"/>
+      <origin xyz="1.42261228e-3 -96.66711845e-3 1.53962525e-3"/>
       <mass value="0.11800000"/>
       <inertia ixx="524.76797677e-6" ixy="16.28790079e-6" ixz="0.26927944e-6" iyy="22.71638836e-6" iyz="-9.50678837e-6" izz="518.76368169e-6"/>
@@ -189,6 +184,5 @@
     </inertial> -->
     <inertial>
-      <!-- <origin xyz="50.33286050e-3 -11.96674465e-3 -0.45712069e-3"/> -->
-      <origin rpy="0 0 0" xyz="0.0557 -0.016 0"/>
+      <origin xyz="50.33286050e-3 -11.96674465e-3 -0.45712069e-3"/>
       <mass value="0.64500000"/>
       <inertia ixx="498.32637694e-6" ixy="43.44106109e-6" ixz="0.22310959e-6" iyy="842.25430695e-6" iyz="-0.01120420e-6" izz="586.98452955e-6"/>
@@ -209,6 +203,5 @@
     </inertial> -->
     <inertial>
-      <!-- <origin xyz="41.97647986e-3 50.28911905e-3 5.24459395e-3"/> -->
-      <origin rpy="0 0 0" xyz="0.031 0.016 0"/>
+      <origin xyz="41.97647986e-3 50.28911905e-3 5.24459395e-3"/>
       <mass value="0.82700000"/>
       <inertia ixx="4027.34061087e-6" ixy="-339.60373031e-6" ixz="-19.19430819e-6" iyy="719.63850817e-6" iyz="-70.69968381e-6" izz="3870.59018254e-6"/>
@@ -235,6 +228,5 @@
     </inertial> -->
     <inertial>
-      <!-- <origin xyz="1.42261242e-3 96.66711821e-3 1.53963358e-3"/> -->
-      <origin rpy="0 0 0" xyz="0.001 0.104 -0.003"/>
+      <origin xyz="1.42261242e-3 96.66711821e-3 1.53963358e-3"/>
       <mass value="0.11800000"/>
       <inertia ixx="524.76797815e-6" ixy="-16.28789980e-6" ixz="0.26927746e-6" iyy="22.71638636e-6" iyz="9.50674532e-6" izz="518.76368492e-6"/>
@@ -289,6 +281,5 @@
     </inertial> -->
     <inertial>
-      <!-- <origin xyz="50.33286050e-3 -11.96674465e-3 -0.45712069e-3"/> -->
-      <origin rpy="0 0 0" xyz="0.0557 -0.016 0"/>
+      <origin xyz="50.33286050e-3 -11.96674465e-3 -0.45712069e-3"/>
       <mass value="0.64500000"/>
       <inertia ixx="498.32637694e-6" ixy="43.44106109e-6" ixz="0.22310959e-6" iyy="842.25430695e-6" iyz="-0.01120420e-6" izz="586.98452955e-6"/>
@@ -309,6 +300,5 @@
     </inertial> -->
     <inertial>
-      <!-- <origin xyz="41.97647986e-3 50.28911905e-3 5.24459395e-3"/> -->
-      <origin rpy="0 0 0" xyz="0.031 0.016 0"/>
+      <origin xyz="41.97647986e-3 50.28911905e-3 5.24459395e-3"/>
       <mass value="0.82700000"/>
       <inertia ixx="4027.34061087e-6" ixy="-339.60373031e-6" ixz="-19.19430819e-6" iyy="719.63850817e-6" iyz="-70.69968381e-6" izz="3870.59018254e-6"/>
@@ -335,6 +325,5 @@
     </inertial> -->
     <inertial>
-      <!-- <origin xyz="1.42261242e-3 96.66711821e-3 1.53963358e-3"/> -->
-      <origin rpy="0 0 0" xyz="0.001 0.104 -0.003"/>
+      <origin xyz="1.42261242e-3 96.66711821e-3 1.53963358e-3"/>
       <mass value="0.11800000"/>
       <inertia ixx="524.76797815e-6" ixy="-16.28789980e-6" ixz="0.26927746e-6" iyy="22.71638636e-6" iyz="9.50674532e-6" izz="518.76368492e-6"/>
@@ -389,6 +378,5 @@
     </inertial> -->
     <inertial>
-      <!-- <origin xyz="50.33286050e-3 11.96674461e-3 0.45712186e-3"/> -->
-      <origin rpy="0 0 0" xyz="0.0557 -0.016 0"/>
+      <origin xyz="50.33286050e-3 11.96674461e-3 0.45712186e-3"/>
       <mass value="0.64500000"/>
       <inertia ixx="498.32637726e-6" ixy="-43.44106123e-6" ixz="-0.22311702e-6" iyy="842.25430777e-6" iyz="-0.01118942e-6" izz="586.98453014e-6"/>
@@ -409,6 +397,5 @@
     </inertial> -->
     <inertial>
-      <!-- <origin xyz="41.97647538e-3 -50.28912232e-3 5.24458524e-3"/> -->
-      <origin rpy="0 0 0" xyz="0.031 -0.016 0"/>
+      <origin xyz="41.97647538e-3 -50.28912232e-3 5.24458524e-3"/>
       <mass value="0.82700000"/>
       <inertia ixx="4027.34053636e-6" ixy="339.60345125e-6" ixz="-19.19423339e-6" iyy="719.63841788e-6" iyz="70.69913102e-6" izz="3870.59006761e-6"/>
@@ -435,6 +422,5 @@
     </inertial> -->
     <inertial>
-      <!-- <origin xyz="1.42261228e-3 -96.66711845e-3 1.53962525e-3"/> -->
-      <origin rpy="0 0 0" xyz="0.001 -0.104 -0.003"/>
+      <origin xyz="1.42261228e-3 -96.66711845e-3 1.53962525e-3"/>
       <mass value="0.11800000"/>
       <inertia ixx="524.76797677e-6" ixy="16.28790079e-6" ixz="0.26927944e-6" iyy="22.71638836e-6" iyz="-9.50678837e-6" izz="518.76368169e-6"/>
