Commit message: robot loading in gazebo with ros2 control (effort controller)

File: mab_description/xacro/silver_badger.gazebo.xacro (robot description, xacro)
@@ -2,59 +2,104 @@
 <robot xmlns:xacro="http://www.ros.org/wiki/xacro">
     <!-- Colors-->
-    <gazebo reference="base_link">
-      <material>Gazebo/Grey</material>
-    </gazebo>
     <gazebo reference="body">
+      <mu1>0.2</mu1>
+      <mu2>0.2</mu2>
       <material>Gazebo/Grey</material>
     </gazebo>
     <gazebo reference="rear">
+      <mu1>0.2</mu1>
+      <mu2>0.2</mu2>
       <material>Gazebo/Grey</material>
     </gazebo>
     <gazebo reference="fr_l0">
+      <mu1>0.2</mu1>
+      <mu2>0.2</mu2>
       <material>Gazebo/Grey</material>
     </gazebo>
     <gazebo reference="fr_l1">
+      <mu1>0.2</mu1>
+      <mu2>0.2</mu2>
       <material>Gazebo/Orange</material>
     </gazebo>
     <gazebo reference="fr_l2">
+      <mu1>0.2</mu1>
+      <mu2>0.2</mu2>
       <material>Gazebo/Grey</material>
     </gazebo>
     <gazebo reference="fr_foot">
+      <mu1>0.6</mu1>
+      <mu2>0.6</mu2>
+      <self_collide>0</self_collide>
+      <kp value="1000000.0"/>
+      <kd value="1.0"/>
       <material>Gazebo/Black</material>
     </gazebo>
     <gazebo reference="fl_l0">
+      <mu1>0.2</mu1>
+      <mu2>0.2</mu2>
       <material>Gazebo/Grey</material>
     </gazebo>
     <gazebo reference="fl_l1">
+      <mu1>0.2</mu1>
+      <mu2>0.2</mu2>
       <material>Gazebo/Orange</material>
     </gazebo>
     <gazebo reference="fl_l2">
+      <mu1>0.2</mu1>
+      <mu2>0.2</mu2>
       <material>Gazebo/Grey</material>
     </gazebo>
     <gazebo reference="fl_foot">
+      <mu1>0.6</mu1>
+      <mu2>0.6</mu2>
+      <self_collide>0</self_collide>
+      <kp value="1000000.0"/>
+      <kd value="1.0"/>
       <material>Gazebo/Black</material>
     </gazebo>
     <gazebo reference="rl_l0">
+      <mu1>0.2</mu1>
+      <mu2>0.2</mu2>
       <material>Gazebo/Grey</material>
     </gazebo>
     <gazebo reference="rl_l1">
+      <mu1>0.2</mu1>
+      <mu2>0.2</mu2>
       <material>Gazebo/Orange</material>
     </gazebo>
     <gazebo reference="rl_l2">
+      <mu1>0.2</mu1>
+      <mu2>0.2</mu2>
       <material>Gazebo/Grey</material>
     </gazebo>
     <gazebo reference="rl_foot">
+      <mu1>0.6</mu1>
+      <mu2>0.6</mu2>
+      <self_collide>0</self_collide>
+      <kp value="1000000.0"/>
+      <kd value="1.0"/>
       <material>Gazebo/Black</material>
     </gazebo>
     <gazebo reference="rr_l0">
+      <mu1>0.2</mu1>
+      <mu2>0.2</mu2>
       <material>Gazebo/Grey</material>
     </gazebo>
     <gazebo reference="rr_l1">
+      <mu1>0.2</mu1>
+      <mu2>0.2</mu2>
       <material>Gazebo/Orange</material>
     </gazebo>
     <gazebo reference="rr_l2">
+      <mu1>0.2</mu1>
+      <mu2>0.2</mu2>
       <material>Gazebo/Grey</material>
     </gazebo>
     <gazebo reference="rr_foot">
+      <mu1>0.6</mu1>
+      <mu2>0.6</mu2>
+      <self_collide>0</self_collide>
+      <kp value="1000000.0"/>
+      <kd value="1.0"/>
       <material>Gazebo/Black</material>
     </gazebo>

File: mab_description/xacro/silver_badger.urdf.xacro (robot description, xacro)
@@ -5,69 +5,26 @@
   </mujoco>
   <!-- Include gazebo elements and colors-->
-  <xacro:include filename="$(find mab_description)/urdf/silver_badger.gazebo.xacro" />
+  <xacro:include filename="$(find mab_description)/xacro/silver_badger.gazebo.xacro" />
   <!-- Import Rviz colors -->
-  <xacro:include filename="$(find mab_description)/urdf/materials.xacro" />
-  <!-- joint limits -->
-  <xacro:property name="fr_j0_limit_lower" value="-1.57"/>
-  <xacro:property name="fr_j0_limit_upper" value="1.57"/>
-  <xacro:property name="fr_j1_limit_lower" value="-1.57"/>
-  <xacro:property name="fr_j1_limit_upper" value="1.57"/>
-  <xacro:property name="fr_j2_limit_lower" value="-2.53"/>
-  <xacro:property name="fr_j2_limit_upper" value="0.0"/>
-  <xacro:property name="fl_j0_limit_lower" value="-1.57"/>
-  <xacro:property name="fl_j0_limit_upper" value="1.57"/>
-  <xacro:property name="fl_j1_limit_lower" value="-1.57"/>
-  <xacro:property name="fl_j1_limit_upper" value="1.57"/>
-  <xacro:property name="fl_j2_limit_lower" value="0.0"/>
-  <xacro:property name="fl_j2_limit_upper" value="2.53"/>
-  <xacro:property name="rl_j0_limit_lower" value="-1.57"/>
-  <xacro:property name="rl_j0_limit_upper" value="1.57"/>
-  <xacro:property name="rl_j1_limit_lower" value="-1.57"/>
-  <xacro:property name="rl_j1_limit_upper" value="1.57"/>
-  <xacro:property name="rl_j2_limit_lower" value="0.0"/>
-  <xacro:property name="rl_j2_limit_upper" value="2.53"/>
-  <xacro:property name="rr_j0_limit_lower" value="-1.57"/>
-  <xacro:property name="rr_j0_limit_upper" value="1.57"/>
-  <xacro:property name="rr_j1_limit_lower" value="-1.57"/>
-  <xacro:property name="rr_j1_limit_upper" value="1.57"/>
-  <xacro:property name="rr_j2_limit_lower" value="-2.53"/>
-  <xacro:property name="rr_j2_limit_upper" value="0.0"/>
-  <!-- max torques per joint -->
-  <xacro:property name="fr_j0_max_effort" value="16"/>
-  <xacro:property name="fr_j1_max_effort" value="16"/>
-  <xacro:property name="fr_j2_max_effort" value="16"/>
-  <xacro:property name="fl_j0_max_effort" value="16"/>
-  <xacro:property name="fl_j1_max_effort" value="16"/>
-  <xacro:property name="fl_j2_max_effort" value="16"/>
-  <xacro:property name="rl_j0_max_effort" value="16"/>
-  <xacro:property name="rl_j1_max_effort" value="16"/>
-  <xacro:property name="rl_j2_max_effort" value="16"/>
-  <xacro:property name="rr_j0_max_effort" value="16"/>
-  <xacro:property name="rr_j1_max_effort" value="16"/>
-  <xacro:property name="rr_j2_max_effort" value="16"/>
-  <!-- max velocities per joint -->
-  <xacro:property name="fr_j0_max_velocity" value="25"/>
-  <xacro:property name="fr_j1_max_velocity" value="25"/>
-  <xacro:property name="fr_j2_max_velocity" value="25"/>
-  <xacro:property name="fl_j0_max_velocity" value="25"/>
-  <xacro:property name="fl_j1_max_velocity" value="25"/>
-  <xacro:property name="fl_j2_max_velocity" value="25"/>
-  <xacro:property name="rl_j0_max_velocity" value="25"/>
-  <xacro:property name="rl_j1_max_velocity" value="25"/>
-  <xacro:property name="rl_j2_max_velocity" value="25"/>
-  <xacro:property name="rr_j0_max_velocity" value="25"/>
-  <xacro:property name="rr_j1_max_velocity" value="25"/>
-  <xacro:property name="rr_j2_max_velocity" value="25"/>
-  <!--
-  ##########################################################
-  ###########             BODY              ################
-  ##########################################################
-  -->
+  <xacro:include filename="$(find mab_description)/xacro/materials.xacro" />
+  <!-- Import control tags-->
+  <xacro:include filename="$(find mab_description)/xacro/control.xacro" />
+  <!-- Include limits-->
+  <xacro:include filename="$(find mab_description)/xacro/limits.xacro" />
+  <!-- Initialize controls-->
+  <xacro:silver_badger_ros2_control/>
+  <!-- BODY -->
   <link name="base_link"/>
   <link name="body">
-    <inertial>
+    <!-- <inertial>
       <origin rpy="0 0 0" xyz="0 0 0"/>
       <mass value="5.423"/>
       <inertia ixx="0.1946" ixy="0" ixz="0" iyy="0.4899" iyz="0" izz="0.6228"/>
+    </inertial> -->
+    <inertial>
+      <!-- <origin xyz="19.23637020e-3 0.65977049e-3 3.38565104e-3"/> -->
+      <origin rpy="0 0 0" xyz="0 0 0"/>
+      <mass value="5.42300000"/>
+      <inertia ixx="21646.56458935e-6" ixy="-46.55756531e-6" ixz="18.07857599e-6" iyy="40703.39489390e-6" iyz="-71.07150002e-6" izz="54721.98086004e-6"/>
     </inertial>
     <visual>
@@ -87,8 +44,14 @@
   </link>
   <link name="rear">
-    <inertial>
+    <!-- <inertial>
       <origin rpy="0 0 0" xyz="-0.038 0.075 0"/>
       <mass value="1.337"/>
       <inertia ixx="0.09" ixy="0" ixz="0" iyy="0.0835" iyz="0" izz="0.1561"/>
+    </inertial> -->
+    <inertial>
+      <!-- <origin xyz="-38.28391582e-3 65.76740154e-3 0.15093929e-3"/> -->
+      <origin rpy="0 0 0" xyz="-0.038 0.075 0"/>
+      <mass value="1.33700000"/>
+      <inertia ixx="1982.84311251e-6" ixy="-36.51038588e-6" ixz="-4.15042187e-6" iyy="4644.92962873e-6" iyz="0.10412770e-6" izz="5097.13064643e-6"/>
     </inertial>
     <visual>
@@ -112,5 +75,5 @@
     <origin rpy="3.14159 0 4.71" xyz="-0.141 -0.0395 0"/>
     <axis xyz="1 0 0"/>
-    <limit effort="48.0" lower="-0.785" upper="0.785" velocity="3.15"/>
+    <limit effort="${sp_j0_max_effort}" lower="${sp_j0_limit_lower}" upper="${sp_j0_limit_upper}" velocity="${sp_j0_max_velocity}"/>
   </joint>
   <joint name="root" type="fixed">
@@ -118,14 +81,16 @@
     <child link="body"/>
   </joint>
-  <!--
-  ##########################################################
-  ###########         LEGS LINKS 0-4        ################
-  ##########################################################
-  -->
+  <!-- LEG LINKS 0-4 -->
   <link name="fr_l0">
-    <inertial>
+    <!-- <inertial>
       <origin rpy="0 0 0" xyz="0.0557 -0.016 0"/>
       <mass value="0.645"/>
       <inertia ixx="0.0052" ixy="0" ixz="0" iyy="0.0093" iyz="0" izz="0.0065"/>
+    </inertial> -->
+    <inertial>
+      <!-- <origin xyz="50.33286050e-3 11.96674461e-3 0.45712186e-3"/> -->
+      <origin rpy="0 0 0" xyz="0.0557 -0.016 0"/>
+      <mass value="0.64500000"/>
+      <inertia ixx="498.32637726e-6" ixy="-43.44106123e-6" ixz="-0.22311702e-6" iyy="842.25430777e-6" iyz="-0.01118942e-6" izz="586.98453014e-6"/>
     </inertial>
     <visual>
@@ -138,8 +103,14 @@
   </link>
   <link name="fr_l1">
-    <inertial>
+    <!-- <inertial>
       <origin rpy="0 0 0" xyz="0.031 -0.016 0"/>
       <mass value="0.827"/>
       <inertia ixx="0.0330" ixy="0" ixz="0" iyy="0.0077" iyz="0" izz="0.0286"/>
+    </inertial> -->
+    <inertial>
+      <!-- <origin xyz="41.97647538e-3 -50.28912232e-3 5.24458524e-3"/> -->
+      <origin rpy="0 0 0" xyz="0.031 -0.016 0"/>
+      <mass value="0.82700000"/>
+      <inertia ixx="4027.34053636e-6" ixy="339.60345125e-6" ixz="-19.19423339e-6" iyy="719.63841788e-6" iyz="70.69913102e-6" izz="3870.59006761e-6"/>
     </inertial>
     <visual>
@@ -158,8 +129,14 @@
   </link>
   <link name="fr_l2">
-    <inertial>
+    <!-- <inertial>
       <origin rpy="0 0 0" xyz="0.001 -0.104 -0.003"/>
       <mass value="0.118"/>
       <inertia ixx="0.0213" ixy="0" ixz="0" iyy="0.0002" iyz="0" izz="0.0212"/>
+    </inertial> -->
+    <inertial>
+      <!-- <origin xyz="1.42261228e-3 -96.66711845e-3 1.53962525e-3"/> -->
+      <origin rpy="0 0 0" xyz="0.001 -0.104 -0.003"/>
+      <mass value="0.11800000"/>
+      <inertia ixx="524.76797677e-6" ixy="16.28790079e-6" ixz="0.26927944e-6" iyy="22.71638836e-6" iyz="-9.50678837e-6" izz="518.76368169e-6"/>
     </inertial>
     <visual>
@@ -206,8 +183,14 @@
   </link>
   <link name="fl_l0">
-    <inertial>
+    <!-- <inertial>
       <origin rpy="0 0 0" xyz="0.0557 -0.016 0"/>
       <mass value="0.645"/>
       <inertia ixx="0.0052" ixy="0" ixz="0" iyy="0.0093" iyz="0" izz="0.0065"/>
+    </inertial> -->
+    <inertial>
+      <!-- <origin xyz="50.33286050e-3 -11.96674465e-3 -0.45712069e-3"/> -->
+      <origin rpy="0 0 0" xyz="0.0557 -0.016 0"/>
+      <mass value="0.64500000"/>
+      <inertia ixx="498.32637694e-6" ixy="43.44106109e-6" ixz="0.22310959e-6" iyy="842.25430695e-6" iyz="-0.01120420e-6" izz="586.98452955e-6"/>
     </inertial>
     <visual>
@@ -220,8 +203,14 @@
   </link>
   <link name="fl_l1">
-    <inertial>
+    <!-- <inertial>
       <origin rpy="0 0 0" xyz="0.031 0.016 0"/>
       <mass value="0.827"/>
       <inertia ixx="0.0330" ixy="0" ixz="0" iyy="0.0077" iyz="0" izz="0.0286"/>
+    </inertial> -->
+    <inertial>
+      <!-- <origin xyz="41.97647986e-3 50.28911905e-3 5.24459395e-3"/> -->
+      <origin rpy="0 0 0" xyz="0.031 0.016 0"/>
+      <mass value="0.82700000"/>
+      <inertia ixx="4027.34061087e-6" ixy="-339.60373031e-6" ixz="-19.19430819e-6" iyy="719.63850817e-6" iyz="-70.69968381e-6" izz="3870.59018254e-6"/>
     </inertial>
     <visual>
@@ -240,8 +229,14 @@
   </link>
   <link name="fl_l2">
-    <inertial>
+    <!-- <inertial>
       <origin rpy="0 0 0" xyz="0.001 0.104 -0.003"/>
       <mass value="0.118"/>
       <inertia ixx="0.0213" ixy="0" ixz="0" iyy="0.0002" iyz="0" izz="0.0212"/>
+    </inertial> -->
+    <inertial>
+      <!-- <origin xyz="1.42261242e-3 96.66711821e-3 1.53963358e-3"/> -->
+      <origin rpy="0 0 0" xyz="0.001 0.104 -0.003"/>
+      <mass value="0.11800000"/>
+      <inertia ixx="524.76797815e-6" ixy="-16.28789980e-6" ixz="0.26927746e-6" iyy="22.71638636e-6" iyz="9.50674532e-6" izz="518.76368492e-6"/>
     </inertial>
     <visual>
@@ -288,8 +283,14 @@
   </link>
   <link name="rl_l0">
-    <inertial>
+    <!-- <inertial>
       <origin rpy="0 0 0" xyz="0.0557 -0.016 0"/>
       <mass value="0.645"/>
       <inertia ixx="0.0052" ixy="0" ixz="0" iyy="0.0093" iyz="0" izz="0.0065"/>
+    </inertial> -->
+    <inertial>
+      <!-- <origin xyz="50.33286050e-3 -11.96674465e-3 -0.45712069e-3"/> -->
+      <origin rpy="0 0 0" xyz="0.0557 -0.016 0"/>
+      <mass value="0.64500000"/>
+      <inertia ixx="498.32637694e-6" ixy="43.44106109e-6" ixz="0.22310959e-6" iyy="842.25430695e-6" iyz="-0.01120420e-6" izz="586.98452955e-6"/>
     </inertial>
     <visual>
@@ -302,8 +303,14 @@
   </link>
   <link name="rl_l1">
-    <inertial>
+    <!-- <inertial>
       <origin rpy="0 0 0" xyz="0.031 0.016 0"/>
       <mass value="0.827"/>
       <inertia ixx="0.0330" ixy="0" ixz="0" iyy="0.0077" iyz="0" izz="0.0286"/>
+    </inertial> -->
+    <inertial>
+      <!-- <origin xyz="41.97647986e-3 50.28911905e-3 5.24459395e-3"/> -->
+      <origin rpy="0 0 0" xyz="0.031 0.016 0"/>
+      <mass value="0.82700000"/>
+      <inertia ixx="4027.34061087e-6" ixy="-339.60373031e-6" ixz="-19.19430819e-6" iyy="719.63850817e-6" iyz="-70.69968381e-6" izz="3870.59018254e-6"/>
     </inertial>
     <visual>
@@ -322,8 +329,14 @@
   </link>
   <link name="rl_l2">
-    <inertial>
+    <!-- <inertial>
       <origin rpy="0 0 0" xyz="0.001 0.104 -0.003"/>
       <mass value="0.118"/>
       <inertia ixx="0.0213" ixy="0" ixz="0" iyy="0.0002" iyz="0" izz="0.0212"/>
+    </inertial> -->
+    <inertial>
+      <!-- <origin xyz="1.42261242e-3 96.66711821e-3 1.53963358e-3"/> -->
+      <origin rpy="0 0 0" xyz="0.001 0.104 -0.003"/>
+      <mass value="0.11800000"/>
+      <inertia ixx="524.76797815e-6" ixy="-16.28789980e-6" ixz="0.26927746e-6" iyy="22.71638636e-6" iyz="9.50674532e-6" izz="518.76368492e-6"/>
     </inertial>
     <visual>
@@ -370,8 +383,14 @@
   </link>
   <link name="rr_l0">
-    <inertial>
+    <!-- <inertial>
       <origin rpy="0 0 0" xyz="0.0557 -0.016 0"/>
       <mass value="0.645"/>
       <inertia ixx="0.0052" ixy="0" ixz="0" iyy="0.0093" iyz="0" izz="0.0065"/>
+    </inertial> -->
+    <inertial>
+      <!-- <origin xyz="50.33286050e-3 11.96674461e-3 0.45712186e-3"/> -->
+      <origin rpy="0 0 0" xyz="0.0557 -0.016 0"/>
+      <mass value="0.64500000"/>
+      <inertia ixx="498.32637726e-6" ixy="-43.44106123e-6" ixz="-0.22311702e-6" iyy="842.25430777e-6" iyz="-0.01118942e-6" izz="586.98453014e-6"/>
     </inertial>
     <visual>
@@ -384,8 +403,14 @@
   </link>
   <link name="rr_l1">
-    <inertial>
+    <!-- <inertial>
       <origin rpy="0 0 0" xyz="0.031 -0.016 0"/>
       <mass value="0.827"/>
       <inertia ixx="0.0330" ixy="0" ixz="0" iyy="0.0077" iyz="0" izz="0.0286"/>
+    </inertial> -->
+    <inertial>
+      <!-- <origin xyz="41.97647538e-3 -50.28912232e-3 5.24458524e-3"/> -->
+      <origin rpy="0 0 0" xyz="0.031 -0.016 0"/>
+      <mass value="0.82700000"/>
+      <inertia ixx="4027.34053636e-6" ixy="339.60345125e-6" ixz="-19.19423339e-6" iyy="719.63841788e-6" iyz="70.69913102e-6" izz="3870.59006761e-6"/>
     </inertial>
     <visual>
@@ -404,8 +429,14 @@
   </link>
   <link name="rr_l2">
-    <inertial>
+    <!-- <inertial>
       <origin rpy="0 0 0" xyz="0.001 -0.104 -0.003"/>
       <mass value="0.118"/>
       <inertia ixx="0.0213" ixy="0" ixz="0" iyy="0.0002" iyz="0" izz="0.0212"/>
+    </inertial> -->
+    <inertial>
+      <!-- <origin xyz="1.42261228e-3 -96.66711845e-3 1.53962525e-3"/> -->
+      <origin rpy="0 0 0" xyz="0.001 -0.104 -0.003"/>
+      <mass value="0.11800000"/>
+      <inertia ixx="524.76797677e-6" ixy="16.28790079e-6" ixz="0.26927944e-6" iyy="22.71638836e-6" iyz="-9.50678837e-6" izz="518.76368169e-6"/>
     </inertial>
     <visual>
@@ -451,9 +482,5 @@
     </collision>
   </link>
-  <!--
-  ##########################################################
-  ###########        LEGS JOINTS 0-4        ################
-  ##########################################################
-  -->
+  <!-- LEG JOINTS 0-4 -->
   <!-- Front Right Leg -->
   <joint armature="0.01" name="fr_j0" type="continuous">
@@ -568,3 +595,4 @@
     <axis xyz="0.0 0 0"/>
   </joint>
+  <!-- <xacro:silver_badger_ros2_control/> -->
 </robot>
