Commit message: integration with policy and custom gazebo plugin

File: mab_description/xacro/silver_badger.gazebo.xacro (robot description, xacro)
@@ -104,9 +104,30 @@
       <material>Gazebo/Black</material>
     </gazebo>
-    <!-- Controller-->
-    <gazebo>
+    <!-- Controllers-->
+    <!-- <gazebo>
       <plugin name="gazebo_ros2_control" filename="libgazebo_ros2_control.so">
         <parameters>$(find mab_gazebo)/config/silver_badger_controller.yaml</parameters>
       </plugin>
+    </gazebo> -->
+    <gazebo>
+      <plugin name="mab_gazebo_plugin" filename="libmab_gazebo_plugin.so"/>
     </gazebo>
+    <!-- Sensors-->
+    <gazebo reference="imu_link">
+      <gravity>true</gravity>
+      <sensor name='imu_sensor' type='imu'>
+          <always_on>1</always_on>
+          <update_rate>1000</update_rate>
+          <visualize>1</visualize>
+          <topic>imu</topic>
+          <plugin name='imu' filename='libgazebo_ros_imu_sensor.so'>
+              <topicName>imu</topicName>
+              <bodyName>imu_sensor_link</bodyName>
+              <updateRateHZ>100.0</updateRateHZ>
+              <xyzOffset>0 0 0</xyzOffset>
+              <rpyOffset>0 0 0</rpyOffset>
+          </plugin>
+          <pose>0 0 0 0 0 0</pose>
+      </sensor>
+  </gazebo>
 </robot>

File: mab_description/xacro/silver_badger.urdf.xacro (robot description, xacro)
@@ -4,4 +4,6 @@
     <compiler balanceinertia="false" discardvisual="false"/>
   </mujoco>
+  <!-- Include IMU-->
+  <xacro:include filename="$(find mab_description)/xacro/imu.xacro" />
   <!-- Include gazebo elements and colors-->
   <xacro:include filename="$(find mab_description)/xacro/silver_badger.gazebo.xacro" />
@@ -68,4 +70,512 @@
     </collision>
   </link>
+  <joint name="root" type="fixed">
+    <parent link="base_link"/>
+    <child link="body"/>
+  </joint>
+  <xacro:imu parent_link="body"/>
+  <!-- LEG LINKS 0-4 -->
+  <link name="fr_l0">
+    <!-- <inertial>
+      <origin rpy="0 0 0" xyz="0.0557 -0.016 0"/>
+      <mass value="0.645"/>
+      <inertia ixx="0.0052" ixy="0" ixz="0" iyy="0.0093" iyz="0" izz="0.0065"/>
+    </inertial> -->
+    <inertial>
+      <origin xyz="50.33286050e-3 11.96674461e-3 0.45712186e-3"/>
+      <mass value="0.64500000"/>
+      <inertia ixx="498.32637726e-6" ixy="-43.44106123e-6" ixz="-0.22311702e-6" iyy="842.25430777e-6" iyz="-0.01118942e-6" izz="586.98453014e-6"/>
+    </inertial>
+    <visual>
+      <origin rpy="0 0 0" xyz="0 0 0"/>
+      <geometry>
+        <mesh filename="package://meshes/hb40/l0r.stl" scale="0.001 0.001 0.001"/>
+      </geometry>
+      <material name="silver"/>
+    </visual>
+  </link>
+  <link name="fr_l1">
+    <!-- <inertial>
+      <origin rpy="0 0 0" xyz="0.031 -0.016 0"/>
+      <mass value="0.827"/>
+      <inertia ixx="0.0330" ixy="0" ixz="0" iyy="0.0077" iyz="0" izz="0.0286"/>
+    </inertial> -->
+    <inertial>
+      <origin xyz="41.97647538e-3 -50.28912232e-3 5.24458524e-3"/>
+      <mass value="0.82700000"/>
+      <inertia ixx="4027.34053636e-6" ixy="339.60345125e-6" ixz="-19.19423339e-6" iyy="719.63841788e-6" iyz="70.69913102e-6" izz="3870.59006761e-6"/>
+    </inertial>
+    <visual>
+      <origin rpy="0 0 0" xyz="0 0 0"/>
+      <geometry>
+        <mesh filename="package://meshes/hb40/l1r.stl" scale="0.001 0.001 0.001"/>
+      </geometry>
+      <material name="orange"/>
+    </visual>
+    <collision>
+      <origin rpy="0 1.57 0" xyz="0.0 0 0"/>
+      <geometry>
+        <cylinder length="0.08" radius="0.05"/>
+      </geometry>
+    </collision>
+  </link>
+  <link name="fr_l2">
+    <!-- <inertial>
+      <origin rpy="0 0 0" xyz="0.001 -0.104 -0.003"/>
+      <mass value="0.118"/>
+      <inertia ixx="0.0213" ixy="0" ixz="0" iyy="0.0002" iyz="0" izz="0.0212"/>
+    </inertial> -->
+    <inertial>
+      <origin xyz="1.42261228e-3 -96.66711845e-3 1.53962525e-3"/>
+      <mass value="0.11800000"/>
+      <inertia ixx="524.76797677e-6" ixy="16.28790079e-6" ixz="0.26927944e-6" iyy="22.71638836e-6" iyz="-9.50678837e-6" izz="518.76368169e-6"/>
+    </inertial>
+    <visual>
+      <origin rpy="0 0 0" xyz="0 0 0"/>
+      <geometry>
+        <mesh filename="package://meshes/hb40/l2r.stl" scale="0.001 0.001 0.001"/>
+      </geometry>
+      <material name="red"/>
+    </visual>
+    <collision>
+      <origin rpy="1.3 0 0" xyz="0 0.01 0.0055"/>
+      <geometry>
+        <cylinder length="0.0625" radius="0.01"/>
+      </geometry>
+      <material name="invisible"/>
+    </collision>
+    <collision>
+      <origin rpy="1.67 0.0 0.05" xyz="0 -0.1 0.005"/>
+      <geometry>
+        <cylinder length="0.2" radius="0.015"/>
+      </geometry>
+      <material name="invisible"/>
+    </collision>
+  </link>
+    <link name="fr_foot">
+    <inertial>
+      <origin rpy="0 0 0" xyz="0.0 0.0 0.0"/>
+      <mass value="0.0"/>
+      <inertia ixx="0.0" ixy="0" ixz="0" iyy="0.0" iyz="0" izz="0.0"/>
+    </inertial>
+    <visual>
+      <origin rpy="0 0 0" xyz="0 0 0"/>
+      <geometry>
+        <sphere radius="0.021"/>
+      </geometry>
+      <material name="black"/>
+    </visual>
+    <collision>
+      <origin rpy="0 0 0" xyz="0 0 0"/>
+      <geometry>
+        <sphere radius="0.02"/>
+      </geometry>
+    </collision>
+  </link>
+  <link name="fl_l0">
+    <!-- <inertial>
+      <origin rpy="0 0 0" xyz="0.0557 -0.016 0"/>
+      <mass value="0.645"/>
+      <inertia ixx="0.0052" ixy="0" ixz="0" iyy="0.0093" iyz="0" izz="0.0065"/>
+    </inertial> -->
+    <inertial>
+      <origin xyz="50.33286050e-3 -11.96674465e-3 -0.45712069e-3"/>
+      <mass value="0.64500000"/>
+      <inertia ixx="498.32637694e-6" ixy="43.44106109e-6" ixz="0.22310959e-6" iyy="842.25430695e-6" iyz="-0.01120420e-6" izz="586.98452955e-6"/>
+    </inertial>
+    <visual>
+      <origin rpy="0 0 0" xyz="0 0 0"/>
+      <geometry>
+        <mesh filename="package://meshes/hb40/l0l.stl" scale="0.001 0.001 0.001"/>
+      </geometry>
+      <material name="silver"/>
+    </visual>
+  </link>
+  <link name="fl_l1">
+    <!-- <inertial>
+      <origin rpy="0 0 0" xyz="0.031 0.016 0"/>
+      <mass value="0.827"/>
+      <inertia ixx="0.0330" ixy="0" ixz="0" iyy="0.0077" iyz="0" izz="0.0286"/>
+    </inertial> -->
+    <inertial>
+      <origin xyz="41.97647986e-3 50.28911905e-3 5.24459395e-3"/>
+      <mass value="0.82700000"/>
+      <inertia ixx="4027.34061087e-6" ixy="-339.60373031e-6" ixz="-19.19430819e-6" iyy="719.63850817e-6" iyz="-70.69968381e-6" izz="3870.59018254e-6"/>
+    </inertial>
+    <visual>
+      <origin rpy="0 0 0" xyz="0 0 0"/>
+      <geometry>
+        <mesh filename="package://meshes/hb40/l1lf.stl" scale="0.001 0.001 0.001"/>
+      </geometry>
+      <material name="orange"/>
+    </visual>
+    <collision>
+      <origin rpy="0 1.57 0" xyz="0.0 0 0"/>
+      <geometry>
+        <cylinder length="0.08" radius="0.05"/>
+      </geometry>
+    </collision>
+  </link>
+  <link name="fl_l2">
+    <!-- <inertial>
+      <origin rpy="0 0 0" xyz="0.001 0.104 -0.003"/>
+      <mass value="0.118"/>
+      <inertia ixx="0.0213" ixy="0" ixz="0" iyy="0.0002" iyz="0" izz="0.0212"/>
+    </inertial> -->
+    <inertial>
+      <origin xyz="1.42261242e-3 96.66711821e-3 1.53963358e-3"/>
+      <mass value="0.11800000"/>
+      <inertia ixx="524.76797815e-6" ixy="-16.28789980e-6" ixz="0.26927746e-6" iyy="22.71638636e-6" iyz="9.50674532e-6" izz="518.76368492e-6"/>
+    </inertial>
+    <visual>
+      <origin rpy="0 0 0" xyz="0 0 0"/>
+      <geometry>
+        <mesh filename="package://meshes/hb40/l2l.stl" scale="0.001 0.001 0.001"/>
+      </geometry>
+      <material name="silver"/>
+    </visual>
+    <collision>
+      <origin rpy="-1.3 0.0 -0.00" xyz="0 -0.01 0.0055"/>
+      <geometry>
+        <cylinder length="0.0625" radius="0.01"/>
+      </geometry>
+      <material name="invisible"/>
+    </collision>
+    <collision>
+      <origin rpy="-1.67 0.0 -0.05" xyz="0 0.1 0.005"/>
+      <geometry>
+        <cylinder length="0.2" radius="0.015"/>
+      </geometry>
+      <material name="invisible"/>
+    </collision>
+  </link>
+  <link name="fl_foot">
+    <inertial>
+      <origin rpy="0 0 0" xyz="0.0 0.0 0.0"/>
+      <mass value="0.0"/>
+      <inertia ixx="0.0" ixy="0" ixz="0" iyy="0.0" iyz="0" izz="0.0"/>
+    </inertial>
+    <visual>
+      <origin rpy="0 0 0" xyz="0 0 0"/>
+      <geometry>
+        <sphere radius="0.021"/>
+      </geometry>
+      <material name="black"/>
+    </visual>
+    <collision>
+      <origin rpy="0 0 0" xyz="0 0 0"/>
+      <geometry>
+        <sphere radius="0.02"/>
+      </geometry>
+    </collision>
+  </link>
+  <link name="rl_l0">
+    <!-- <inertial>
+      <origin rpy="0 0 0" xyz="0.0557 -0.016 0"/>
+      <mass value="0.645"/>
+      <inertia ixx="0.0052" ixy="0" ixz="0" iyy="0.0093" iyz="0" izz="0.0065"/>
+    </inertial> -->
+    <inertial>
+      <origin xyz="50.33286050e-3 -11.96674465e-3 -0.45712069e-3"/>
+      <mass value="0.64500000"/>
+      <inertia ixx="498.32637694e-6" ixy="43.44106109e-6" ixz="0.22310959e-6" iyy="842.25430695e-6" iyz="-0.01120420e-6" izz="586.98452955e-6"/>
+    </inertial>
+    <visual>
+      <origin rpy="0 0 0" xyz="0 0 0"/>
+      <geometry>
+        <mesh filename="package://meshes/hb40/l0l.stl" scale="0.001 0.001 0.001"/>
+      </geometry>
+      <material name="silver"/>
+    </visual>
+  </link>
+  <link name="rl_l1">
+    <!-- <inertial>
+      <origin rpy="0 0 0" xyz="0.031 0.016 0"/>
+      <mass value="0.827"/>
+      <inertia ixx="0.0330" ixy="0" ixz="0" iyy="0.0077" iyz="0" izz="0.0286"/>
+    </inertial> -->
+    <inertial>
+      <origin xyz="41.97647986e-3 50.28911905e-3 5.24459395e-3"/>
+      <mass value="0.82700000"/>
+      <inertia ixx="4027.34061087e-6" ixy="-339.60373031e-6" ixz="-19.19430819e-6" iyy="719.63850817e-6" iyz="-70.69968381e-6" izz="3870.59018254e-6"/>
+    </inertial>
+    <visual>
+      <origin rpy="0 0 0" xyz="0 0 0"/>
+      <geometry>
+        <mesh filename="package://meshes/hb40/l1lf.stl" scale="0.001 0.001 0.001"/>
+      </geometry>
+      <material name="orange"/>
+    </visual>
+    <collision>
+      <origin rpy="0 1.57 0" xyz="0.0 0 0"/>
+      <geometry>
+        <cylinder length="0.08" radius="0.05"/>
+      </geometry>
+    </collision>
+  </link>
+  <link name="rl_l2">
+    <!-- <inertial>
+      <origin rpy="0 0 0" xyz="0.001 0.104 -0.003"/>
+      <mass value="0.118"/>
+      <inertia ixx="0.0213" ixy="0" ixz="0" iyy="0.0002" iyz="0" izz="0.0212"/>
+    </inertial> -->
+    <inertial>
+      <origin xyz="1.42261242e-3 96.66711821e-3 1.53963358e-3"/>
+      <mass value="0.11800000"/>
+      <inertia ixx="524.76797815e-6" ixy="-16.28789980e-6" ixz="0.26927746e-6" iyy="22.71638636e-6" iyz="9.50674532e-6" izz="518.76368492e-6"/>
+    </inertial>
+    <visual>
+      <origin rpy="0 0 0" xyz="0 0 0"/>
+      <geometry>
+        <mesh filename="package://meshes/hb40/l2l.stl" scale="0.001 0.001 0.001"/>
+      </geometry>
+      <material name="silver"/>
+    </visual>
+    <collision>
+      <origin rpy="-1.3 0 0" xyz="0 -0.01 0.0055"/>
+      <geometry>
+        <cylinder length="0.0625" radius="0.01"/>
+      </geometry>
+      <material name="invisible"/>
+    </collision>
+    <collision>
+      <origin rpy="-1.67 0.0 -0.05" xyz="0 0.1 0.005"/>
+      <geometry>
+        <cylinder length="0.2" radius="0.015"/>
+        <material name="invisible"/>
+      </geometry>
+    </collision>
+  </link>
+  <link name="rl_foot">
+    <inertial>
+      <origin rpy="0 0 0" xyz="0.0 0.0 0.0"/>
+      <mass value="0.0"/>
+      <inertia ixx="0.0" ixy="0" ixz="0" iyy="0.0" iyz="0" izz="0.0"/>
+    </inertial>
+    <visual>
+      <origin rpy="0 0 0" xyz="0 0 0"/>
+      <geometry>
+        <sphere radius="0.021"/>
+      </geometry>
+      <material name="black"/>
+    </visual>
+    <collision>
+      <origin rpy="0 0 0" xyz="0 0 0"/>
+      <geometry>
+        <sphere radius="0.02"/>
+      </geometry>
+    </collision>
+  </link>
+  <link name="rr_l0">
+    <!-- <inertial>
+      <origin rpy="0 0 0" xyz="0.0557 -0.016 0"/>
+      <mass value="0.645"/>
+      <inertia ixx="0.0052" ixy="0" ixz="0" iyy="0.0093" iyz="0" izz="0.0065"/>
+    </inertial> -->
+    <inertial>
+      <origin xyz="50.33286050e-3 11.96674461e-3 0.45712186e-3"/>
+      <mass value="0.64500000"/>
+      <inertia ixx="498.32637726e-6" ixy="-43.44106123e-6" ixz="-0.22311702e-6" iyy="842.25430777e-6" iyz="-0.01118942e-6" izz="586.98453014e-6"/>
+    </inertial>
+    <visual>
+      <origin rpy="0 0 0" xyz="0 0 0"/>
+      <geometry>
+        <mesh filename="package://meshes/hb40/l0r.stl" scale="0.001 0.001 0.001"/>
+      </geometry>
+      <material name="silver"/>
+    </visual>
+  </link>
+  <link name="rr_l1">
+    <!-- <inertial>
+      <origin rpy="0 0 0" xyz="0.031 -0.016 0"/>
+      <mass value="0.827"/>
+      <inertia ixx="0.0330" ixy="0" ixz="0" iyy="0.0077" iyz="0" izz="0.0286"/>
+    </inertial> -->
+    <inertial>
+      <origin xyz="41.97647538e-3 -50.28912232e-3 5.24458524e-3"/>
+      <mass value="0.82700000"/>
+      <inertia ixx="4027.34053636e-6" ixy="339.60345125e-6" ixz="-19.19423339e-6" iyy="719.63841788e-6" iyz="70.69913102e-6" izz="3870.59006761e-6"/>
+    </inertial>
+    <visual>
+      <origin rpy="0 0 0" xyz="0 0 0"/>
+      <geometry>
+        <mesh filename="package://meshes/hb40/l1r.stl" scale="0.001 0.001 0.001"/>
+      </geometry>
+      <material name="orange"/>
+    </visual>
+    <collision>
+      <origin rpy="0 1.57 0" xyz="0.0 0 0"/>
+      <geometry>
+        <cylinder length="0.08" radius="0.05"/>
+      </geometry>
+    </collision>
+  </link>
+  <link name="rr_l2">
+    <!-- <inertial>
+      <origin rpy="0 0 0" xyz="0.001 -0.104 -0.003"/>
+      <mass value="0.118"/>
+      <inertia ixx="0.0213" ixy="0" ixz="0" iyy="0.0002" iyz="0" izz="0.0212"/>
+    </inertial> -->
+    <inertial>
+      <origin xyz="1.42261228e-3 -96.66711845e-3 1.53962525e-3"/>
+      <mass value="0.11800000"/>
+      <inertia ixx="524.76797677e-6" ixy="16.28790079e-6" ixz="0.26927944e-6" iyy="22.71638836e-6" iyz="-9.50678837e-6" izz="518.76368169e-6"/>
+    </inertial>
+    <visual>
+      <origin rpy="0 0 0" xyz="0 0 0"/>
+      <geometry>
+        <mesh filename="package://meshes/hb40/l2r.stl" scale="0.001 0.001 0.001"/>
+      </geometry>
+      <material name="silver"/>
+    </visual>
+    <collision>
+      <origin rpy="1.3 0.0 0" xyz="0 0.01 0.0055"/>
+      <geometry>
+        <cylinder length="0.0625" radius="0.01"/>
+        <material name="invisible"/>
+      </geometry>
+    </collision>
+    <collision>
+      <origin rpy="1.67 0.0 0.05" xyz="0 -0.1 0.005"/>
+      <geometry>
+        <cylinder length="0.2" radius="0.015"/>
+        <material name="invisible"/>
+      </geometry>
+    </collision>
+  </link>
+  <link name="rr_foot">
+    <inertial>
+      <origin rpy="0 0 0" xyz="0.0 0.0 0.0"/>
+      <mass value="0.0"/>
+      <inertia ixx="0.0" ixy="0" ixz="0" iyy="0.0" iyz="0" izz="0.0"/>
+    </inertial>
+    <visual>
+      <origin rpy="0 0 0" xyz="0 0 0"/>
+      <geometry>
+        <sphere radius="0.021"/>
+      </geometry>
+      <material name="black"/>
+    </visual>
+    <collision>
+      <origin rpy="0 0 0" xyz="0 0 0"/>
+      <geometry>
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
Commit message: added realsense camera into gazebo, yet to set correct position

File: mab_description/xacro/silver_badger.gazebo.xacro (robot description, xacro)
@@ -131,3 +131,19 @@
       </sensor>
   </gazebo>
+  <!-- Realsense Camera-->
+  <!-- <gazebo>
+    <plugin name="realsense_camera" filename="librealsense_gazebo_plugin.so"/>
+      <camera_name>depth_camera</camera_name>
+      <depth_topic>/camera/depth/image_raw</depth_topic>
+      <color_topic>/camera/color/image_raw</color_topic>
+      <infrared1_topic>/camera/infra1/image_raw</infrared1_topic>
+      <infrared2_topic>/camera/infra2/image_raw</infrared2_topic>
+      <depth_camera_info_topic>/camera/depth/camera_info</depth_camera_info_topic>
+      <color_camera_info_topic>/camera/color/camera_info</color_camera_info_topic>
+      <infrared1_camera_info_topic>/camera/infra1/camera_info</infrared1_camera_info_topic>
+      <infrared2_camera_info_topic>/camera/infra2/camera_info</infrared2_camera_info_topic>
+      <pointcloud_topic>/camera/depth/points</pointcloud_topic>
+      <pointcloud_cutoff>0.5</pointcloud_cutoff>
+      <range_max>4.0</range_max>
+  </gazebo> -->
 </robot>

File: mab_description/xacro/silver_badger.urdf.xacro (robot description, xacro)
@@ -16,4 +16,7 @@
   <!-- Initialize controls-->
   <xacro:silver_badger_ros2_control/>
+  <!-- Initialize camera-->
+  <xacro:include filename="$(find mab_description)/xacro/camera.xacro"/>
+  <xacro:realsense2_camera parent="base_link" name="d435_camera"/>
   <!-- BODY -->
   <link name="base_link"/>
@@ -75,4 +78,20 @@
   </joint>
   <xacro:imu parent_link="body"/>
+  <!-- <sensor_d435 parent="base_link"/> -->
+  <!-- <link name="realsense_link">
+    <visual>
+      <geometry>
+        <box size="0.1 0.1 0.1"/>
+      </geometry>
+      <material>
+        <color rgba="0 1 0 1"/>
+      </material>
+    </visual>
+  </link>
+  <joint name="realsense_joint" type="fixed">
+    <parent link="base_link"/>
+    <child link="realsense_link"/>
+    <origin xyz="0 0 1.0" rpy="0 0 0"/>
+  </joint> -->
   <!-- LEG LINKS 0-4 -->
   <link name="fr_l0">
