Commit message: stable version with rtabmap_slam

File: mab_description/xacro/camera.xacro (robot description, xacro)
@@ -57,5 +57,5 @@
         <xacro:property name="infrared1_optical_frame" value="${name}_infra1_frame" />
         <xacro:property name="infrared2_optical_frame" value="${name}_infra2_frame" />
-        <xacro:property name="publish_pointcloud" value="true" />
+        <xacro:property name="publish_pointcloud" value="false" />
         <!-- Gazebo stuff for realsense-->
         <!-- Load parameters to model's main link-->
@@ -102,6 +102,6 @@
                     <horizontal_fov>${85.2*deg_to_rad}</horizontal_fov>
                     <image>
-                        <width>1280</width>
-                        <height>720</height>
+                        <width>640</width>
+                        <height>480</height>
                         <format>L_INT8</format>
                     </image>
@@ -117,5 +117,5 @@
                 </camera>
                 <always_on>1</always_on>
-                <update_rate>90</update_rate>
+                <update_rate>0</update_rate>
                 <visualize>0</visualize>
             </sensor>
@@ -124,6 +124,6 @@
                     <horizontal_fov>${85.2*deg_to_rad}</horizontal_fov>
                     <image>
-                        <width>1280</width>
-                        <height>720</height>
+                        <width>640</width>
+                        <height>480</height>
                         <format>L_INT8</format>
                     </image>
@@ -139,5 +139,5 @@
                 </camera>
                 <always_on>1</always_on>
-                <update_rate>90</update_rate>
+                <update_rate>0</update_rate>
                 <visualize>0</visualize>
             </sensor>
@@ -169,5 +169,5 @@
                 <depthUpdateRate>30.0</depthUpdateRate>
                 <colorUpdateRate>30.0</colorUpdateRate>
-                <infraredUpdateRate>30.0</infraredUpdateRate>
+                <infraredUpdateRate>0.0</infraredUpdateRate>
                 <depthTopicName>${topics_ns}/depth/image_raw</depthTopicName>
                 <depthCameraInfoTopicName>${topics_ns}/depth/camera_info</depthCameraInfoTopicName>

File: mab_description/xacro/silver_badger.gazebo.xacro (robot description, xacro)
@@ -124,5 +124,5 @@
       <sensor name='imu_sensor' type='imu'>
           <always_on>1</always_on>
-          <update_rate>1000</update_rate>
+          <update_rate>20</update_rate>
           <visualize>1</visualize>
           <topic>imu</topic>
@@ -130,5 +130,5 @@
               <topicName>imu</topicName>
               <bodyName>imu_sensor_link</bodyName>
-              <updateRateHZ>1000.0</updateRateHZ>
+              <updateRateHZ>20.0</updateRateHZ>
               <xyzOffset>0 0 0</xyzOffset>
               <rpyOffset>0 0 0</rpyOffset>

Commit message: new changes with laser stabilization

File: mab_description/xacro/camera.xacro (robot description, xacro)
@@ -37,11 +37,9 @@
                 <inertia ixx="0" ixy="0" ixz="0" iyy="0" iyz="0" izz="0" />
             </inertial>
-            <visual>
-                <origin rpy="${d435_cam_roll} 0 0" xyz="${d435_cam_x} ${d435_cam_y} ${d435_cam_z}" />
-            </visual>
         </link>
         <joint name="camera_image_joint" type="fixed">
             <parent link="${parent}"/>
             <child link="camera_image_link"/>
+            <!-- <origin rpy="0 0 0" xyz="${d435_cam_x} ${d435_cam_y} ${d435_cam_z}" /> -->
             <origin rpy="${d435_cam_roll} 0 0" xyz="${d435_cam_x} ${d435_cam_y} ${d435_cam_z}" />
         </joint>
@@ -99,5 +97,5 @@
                 </camera>
                 <always_on>1</always_on>
-                <update_rate>90</update_rate>
+                <update_rate>60</update_rate>
                 <visualize>1</visualize>
             </sensor>
@@ -174,7 +172,7 @@
                 <prefix>${camera_name}</prefix>
                 <depthUpdateRate>90.0</depthUpdateRate>
-                <colorUpdateRate>90.0</colorUpdateRate>
+                <colorUpdateRate>60.0</colorUpdateRate>
                 <infraredUpdateRate>0.0</infraredUpdateRate>
-                <depthTopicName>${topics_ns}/depth/image_raw</depthTopicName>
+                <depthTopicName>${topics_ns}/depth/image_rect_raw</depthTopicName>
                 <depthCameraInfoTopicName>${topics_ns}/depth/camera_info</depthCameraInfoTopicName>
                 <colorTopicName>${topics_ns}/color/image_raw</colorTopicName>

File: mab_description/xacro/silver_badger.urdf.xacro (robot description, xacro)
@@ -7,5 +7,6 @@
   <xacro:include filename="$(find mab_description)/xacro/imu.xacro" />
   <!-- Include gazebo elements and colors-->
-  <xacro:include filename="$(find mab_description)/xacro/silver_badger.gazebo.xacro" />
+  <xacro:include filename="$(find mab_description)/xacro/gazebo.xacro" />
+  <xacro:gazebo_simulation robot="silver_badger"/>
   <!-- Import Rviz colors -->
   <xacro:include filename="$(find mab_description)/xacro/materials.xacro" />
@@ -78,14 +79,4 @@
     <child link="body"/>
   </joint>
-  <!-- <link name="map"/>
-  <joint name="map_root" type="floating">
-    <parent link="base_link"/>
-    <child link="map"/>
-  </joint> -->
-  <!-- <link name="odom"/>
-  <joint name="odom_root" type="fixed">
-    <parent link="base_link"/>
-    <child link="odom"/>
-  </joint> -->
   <!-- Setup camera mount-->
   <xacro:realsense2_camera_mount parent="body"/>
