Commit message: all robots walk

File: robots/a1_description/urdf/a1.urdf (robot description, URDF)
Before this commit: robot a1, 23 links, 22 joints
Links:
- link FL_calf: mass 0.166 -> 0.151
- link FL_hip: mass 0.696 -> 0.595
- link FL_thigh: mass 1.013 -> 0.888
- link FR_calf: mass 0.166 -> 0.151
- link FR_hip: mass 0.696 -> 0.595
- link FR_thigh: mass 1.013 -> 0.888
- link RL_calf: mass 0.166 -> 0.151
- link RL_hip: mass 0.696 -> 0.595
- link RL_thigh: mass 1.013 -> 0.888
- link RR_calf: mass 0.166 -> 0.151
- link RR_hip: mass 0.696 -> 0.595
- link RR_thigh: mass 1.013 -> 0.888
Joints:
- joint FL_calf_joint: limit lower=-2.69653369433 upper=-0.916297857297 effort=33.5 velocity=21 -> lower=-2.6965336943312392 upper=-0.9162978572970231 effort=33.5 velocity=21
- joint FL_hip_joint: limit lower=-0.802851455917 upper=0.802851455917 effort=33.5 velocity=21 -> lower=-0.8028514559173915 upper=0.8028514559173915 effort=33.5 velocity=21
- joint FL_thigh_joint: limit lower=-1.0471975512 upper=4.18879020479 effort=33.5 velocity=21 -> lower=-1.0471975511965976 upper=4.1887902047863905 effort=33.5 velocity=21
- joint FR_calf_joint: axis 0 1 0 -> 0 -1 0; limit lower=-2.69653369433 upper=-0.916297857297 effort=33.5 velocity=21 -> lower=0.9162978572970231 upper=2.6965336943312392 effort=33.5 velocity=21
- joint FR_hip_joint: limit lower=-0.802851455917 upper=0.802851455917 effort=33.5 velocity=21 -> lower=-0.8028514559173915 upper=0.8028514559173915 effort=33.5 velocity=21
- joint FR_thigh_joint: axis 0 1 0 -> 0 -1 0; limit lower=-1.0471975512 upper=4.18879020479 effort=33.5 velocity=21 -> lower=-4.1887902047863905 upper=1.0471975511965976 effort=33.5 velocity=21
- joint RL_calf_joint: limit lower=-2.69653369433 upper=-0.916297857297 effort=33.5 velocity=21 -> lower=-2.6965336943312392 upper=-0.9162978572970231 effort=33.5 velocity=21
- joint RL_hip_joint: axis 1 0 0 -> -1 0 0; limit lower=-0.802851455917 upper=0.802851455917 effort=33.5 velocity=21 -> lower=-0.8028514559173915 upper=0.8028514559173915 effort=33.5 velocity=21
- joint RL_thigh_joint: limit lower=-1.0471975512 upper=4.18879020479 effort=33.5 velocity=21 -> lower=-1.0471975511965976 upper=4.1887902047863905 effort=33.5 velocity=21
- joint RR_calf_joint: axis 0 1 0 -> 0 -1 0; limit lower=-2.69653369433 upper=-0.916297857297 effort=33.5 velocity=21 -> lower=0.9162978572970231 upper=2.6965336943312392 effort=33.5 velocity=21
- joint RR_hip_joint: axis 1 0 0 -> -1 0 0; limit lower=-0.802851455917 upper=0.802851455917 effort=33.5 velocity=21 -> lower=-0.8028514559173915 upper=0.8028514559173915 effort=33.5 velocity=21
- joint RR_thigh_joint: axis 0 1 0 -> 0 -1 0; limit lower=-1.0471975512 upper=4.18879020479 effort=33.5 velocity=21 -> lower=-4.1887902047863905 upper=1.0471975511965976 effort=33.5 velocity=21

File: robots/a1_description/xacro/gazebo.xacro (robot description, xacro)
@@ -43,5 +43,5 @@
             <visualize>true</visualize>
             <topic>__default_topic__</topic>
-            <plugin filename="libgazebo_ros_imu_sensor.so" name="imu_plugin">
+            <plugin filename="libgazebo_ros_imu_sensor.so" name="imu">
                 <topicName>trunk_imu</topicName>
                 <bodyName>imu_link</bodyName>
@@ -121,4 +121,10 @@
         </visual>
     </gazebo>
+    <!-- Gazebo neural control plugin -->
+    <gazebo>
+      <plugin name="unitree_gazebo_plugin" filename="libunitree_control.so">
+        <robot>a1</robot>
+      </plugin>
+    </gazebo>
     <gazebo reference="base">
         <material>Gazebo/Green</material>

File: robots/go1_description/urdf/go1.urdf (robot description, URDF)
Before this commit: robot go1, 46 links, 45 joints
Links:
- link FL_calf_rotor: geometry visual cylinder length=0.02 radius=0.035
- link FL_hip_rotor: geometry visual cylinder length=0.02 radius=0.035
- link FL_thigh_rotor: geometry visual cylinder length=0.02 radius=0.035
- link FR_calf_rotor: geometry visual cylinder length=0.02 radius=0.035
- link FR_hip_rotor: geometry visual cylinder length=0.02 radius=0.035
- link FR_thigh_rotor: geometry visual cylinder length=0.02 radius=0.035
- link RL_calf_rotor: geometry visual cylinder length=0.02 radius=0.035
- link RL_hip_rotor: geometry visual cylinder length=0.02 radius=0.035
- link RL_thigh_rotor: geometry visual cylinder length=0.02 radius=0.035
- link RR_calf_rotor: geometry visual cylinder length=0.02 radius=0.035
- link RR_hip_rotor: geometry visual cylinder length=0.02 radius=0.035
- link RR_thigh_rotor: geometry visual cylinder length=0.02 radius=0.035
Joints:
- joint FR_calf_joint: axis 0 1 0 -> 0 -1 0; limit lower=-2.818 upper=-0.888 effort=35.55 velocity=20.06 -> lower=0.888 upper=2.818 effort=35.55 velocity=20.06
- joint FR_thigh_joint: axis 0 1 0 -> 0 -1 0; limit lower=-0.686 upper=4.501 effort=23.7 velocity=30.1 -> lower=-4.501 upper=0.686 effort=23.7 velocity=30.1
- joint RL_hip_joint: axis 1 0 0 -> -1 0 0
- joint RR_calf_joint: axis 0 1 0 -> 0 -1 0; limit lower=-2.818 upper=-0.888 effort=35.55 velocity=20.06 -> lower=0.888 upper=2.818 effort=35.55 velocity=20.06
- joint RR_hip_joint: axis 1 0 0 -> -1 0 0
- joint RR_thigh_joint: axis 0 1 0 -> 0 -1 0; limit lower=-0.686 upper=4.501 effort=23.7 velocity=30.1 -> lower=-4.501 upper=0.686 effort=23.7 velocity=30.1

File: robots/go1_description/xacro/gazebo.xacro (robot description, xacro)
@@ -43,5 +43,5 @@
             <visualize>true</visualize>
             <topic>__default_topic__</topic>
-            <plugin filename="libgazebo_ros_imu_sensor.so" name="imu_plugin">
+            <plugin filename="libgazebo_ros_imu_sensor.so" name="imu">
                 <topicName>trunk_imu</topicName>
                 <bodyName>imu_link</bodyName>
@@ -233,4 +233,9 @@
         </visual>
     </gazebo>
+    <gazebo>
+      <plugin name="unitree_gazebo_plugin" filename="libunitree_control.so">
+        <robot>go1</robot>
+      </plugin>
+    </gazebo>
     <gazebo reference="base">
         <material>Gazebo/Green</material>

File: robots/go2_description/urdf/go2.urdf (robot description, URDF)
Before this commit: robot go2, 31 links, 30 joints
Joints:
- joint FR_calf_joint: axis 0 1 0 -> 0 -1 0; limit lower=-2.7227 upper=-0.83776 effort=35.55 velocity=20.06 -> lower=0.83776 upper=2.7227 effort=35.55 velocity=20.06
- joint FR_thigh_joint: axis 0 1 0 -> 0 -1 0; limit lower=-1.5708 upper=3.4907 effort=23.7 velocity=30.1 -> lower=-3.4907 upper=1.5708 effort=23.7 velocity=30.1
- joint RL_hip_joint: axis 1 0 0 -> -1 0 0
- joint RR_calf_joint: axis 0 1 0 -> 0 -1 0; limit lower=-2.7227 upper=-0.83776 effort=35.55 velocity=20.06 -> lower=0.83776 upper=2.7227 effort=35.55 velocity=20.06
- joint RR_hip_joint: axis 1 0 0 -> -1 0 0
- joint RR_thigh_joint: axis 0 1 0 -> 0 -1 0; limit lower=-1.5708 upper=3.4907 effort=23.7 velocity=30.1 -> lower=-3.4907 upper=1.5708 effort=23.7 velocity=30.1

File: robots/go2_description/xacro/gazebo.xacro (robot description, xacro)
@@ -42,5 +42,5 @@
             <visualize>true</visualize>
             <topic>__default_topic__</topic>
-            <plugin filename="libgazebo_ros_imu_sensor.so" name="imu_plugin">
+            <plugin filename="libgazebo_ros_imu_sensor.so" name="imu">
                 <topicName>trunk_imu</topicName>
                 <bodyName>imu_link</bodyName>
@@ -120,4 +120,10 @@
         </visual>
     </gazebo>
+    <!-- Gazebo neural control plugin -->
+    <gazebo>
+      <plugin name="unitree_gazebo_plugin" filename="libunitree_control.so">
+        <robot>go2</robot>
+      </plugin>
+    </gazebo>
     <gazebo reference="base">
         <turnGravityOff>false</turnGravityOff>

Commit message: general updates

File: robots/a1_description/urdf/a1.urdf (robot description, URDF)
Before this commit: robot a1, 39 links, 38 joints
Joints:
- joint camera_image_joint: origin xyz=0.320755 5.3e-05 0.068583 rpy=-1.5707963267948966 0 0 -> xyz=0.370755 5.3e-05 0.068583 rpy=0.0 0 0
- joint d435i_camera_joint: origin xyz=0.30585500000000004 -0.012447000000000001 0.068583 rpy=-1.5707963267948966 0 0 -> xyz=0.35585500000000003 -0.012447000000000001 0.068583 rpy=0.0 0 0
- joint laser_joint: origin xyz=0 0 0 rpy=1.5707963267948966 0 0 -> xyz=0 0 0 rpy=-0.0 0 0

File: robots/a1_description/xacro/camera.xacro (robot description, xacro)
@@ -19,9 +19,9 @@
         <xacro:property name="d435_cam_depth_pz" value="${d435_cam_height/2}"/>
         <!-- Camera position in 3D-->
-        <xacro:property name="d435_cam_x" value="0.320755"/>
+        <xacro:property name="d435_cam_x" value="0.370755"/>
         <xacro:property name="d435_cam_y" value="0.000053"/>
         <xacro:property name="d435_cam_z" value="0.068583"/>
-        <xacro:property name="d435_cam_roll" value="${-M_PI/2}"/>
-        <!-- <xacro:property name="d435_cam_roll" value="0"/> -->
+        <!-- <xacro:property name="d435_cam_roll" value="${-M_PI/2}"/> -->
+        <xacro:property name="d435_cam_roll" value="0.0"/>
         <!-- Initialize camera-->
         <xacro:include filename="$(find realsense2_description)/urdf/_d435i.urdf.xacro"/>

File: robots/go1_description/urdf/go1.urdf (robot description, URDF)
Before this commit: robot go1, 62 links, 61 joints
Joints:
- joint camera_image_joint: origin xyz=0.330755 5.3e-05 0.068583 rpy=-1.5707963267948966 0 0 -> xyz=0.370755 5.3e-05 0.068583 rpy=0.0 0 0
- joint d435i_camera_joint: origin xyz=0.31585500000000005 -0.012447000000000001 0.068583 rpy=-1.5707963267948966 0 0 -> xyz=0.35585500000000003 -0.012447000000000001 0.068583 rpy=0.0 0 0
- joint laser_joint: origin xyz=0 0 0 rpy=1.5707963267948966 0 0 -> xyz=0 0 0 rpy=-0.0 0 0

File: robots/go1_description/xacro/camera.xacro (robot description, xacro)
@@ -19,9 +19,9 @@
         <xacro:property name="d435_cam_depth_pz" value="${d435_cam_height/2}"/>
         <!-- Camera position in 3D-->
-        <xacro:property name="d435_cam_x" value="0.330755"/>
+        <xacro:property name="d435_cam_x" value="0.370755"/>
         <xacro:property name="d435_cam_y" value="0.000053"/>
         <xacro:property name="d435_cam_z" value="0.068583"/>
-        <xacro:property name="d435_cam_roll" value="${-M_PI/2}"/>
-        <!-- <xacro:property name="d435_cam_roll" value="0"/> -->
+        <!-- <xacro:property name="d435_cam_roll" value="${-M_PI/2}"/> -->
+        <xacro:property name="d435_cam_roll" value="0.0"/>
         <!-- Initialize camera-->
         <xacro:include filename="$(find realsense2_description)/urdf/_d435i.urdf.xacro"/>

File: robots/go2_description/urdf/go2.urdf (robot description, URDF)
Before this commit: robot go2, 47 links, 46 joints
Joints:
- joint camera_image_joint: origin xyz=0.370755 5.3e-05 0.068583 rpy=-1.5707963267948966 0 0 -> xyz=0.370755 5.3e-05 0.03 rpy=0.0 0 0
- joint d435i_camera_joint: origin xyz=0.35585500000000003 -0.012447000000000001 0.068583 rpy=-1.5707963267948966 0 0 -> xyz=0.35585500000000003 -0.012447000000000001 0.03 rpy=0.0 0 0
- joint laser_joint: origin xyz=0 0 0 rpy=1.5707963267948966 0 0 -> xyz=0 0 0 rpy=-0.0 0 0

File: robots/go2_description/xacro/camera.xacro (robot description, xacro)
@@ -21,12 +21,13 @@
         <xacro:property name="d435_cam_x" value="0.370755"/>
         <xacro:property name="d435_cam_y" value="0.000053"/>
-        <xacro:property name="d435_cam_z" value="0.068583"/>
-        <xacro:property name="d435_cam_roll" value="${-M_PI/2}"/>
-        <!-- <xacro:property name="d435_cam_roll" value="0"/> -->
+        <xacro:property name="d435_cam_z" value="0.030000"/>
+        <!-- <xacro:property name="d435_cam_z" value="0.068583"/> -->
+        <!-- <xacro:property name="d435_cam_roll" value="${-M_PI/2}"/> -->
+        <xacro:property name="d435_cam_roll" value="0.0"/>
         <!-- Initialize camera-->
         <xacro:include filename="$(find realsense2_description)/urdf/_d435i.urdf.xacro"/>
         <xacro:sensor_d435i parent="${parent}" name="${name}" use_nominal_extrinsics="true">
             <!-- <origin xyz="${0.290755-d435_mesh_x_offset-d435_zero_depth_to_glass - d435_glass_to_front} ${0.000053-d435_cam_depth_pz} ${0.068583}" rpy="${0} 0 0"/> -->
-            <origin xyz="${d435_cam_x-d435_mesh_x_offset-d435_zero_depth_to_glass - d435_glass_to_front} ${0.000053-d435_cam_depth_pz} ${0.068583}" rpy="${d435_cam_roll} 0 0"/>
+            <origin xyz="${d435_cam_x-d435_mesh_x_offset-d435_zero_depth_to_glass - d435_glass_to_front} ${d435_cam_y-d435_cam_depth_pz} ${d435_cam_z}" rpy="${d435_cam_roll} 0 0"/>
         </xacro:sensor_d435i>
         <!-- Link for camera image and gazebe plugin-->

Commit message: Updates and clean up

File: robots/a1_description/urdf/a1.urdf (robot description, URDF)
Before this commit: robot a1, 39 links, 38 joints
Joints:
- joint camera_image_joint: origin xyz=0.370755 5.3e-05 0.068583 rpy=0.0 0 0 -> xyz=0.270755 5.3e-05 0.01 rpy=0.0 0 0
- joint d435i_camera_joint: origin xyz=0.35585500000000003 -0.012447000000000001 0.068583 rpy=0.0 0 0 -> xyz=0.25585500000000005 -0.012447000000000001 0.01 rpy=0.0 0 0

File: robots/a1_description/xacro/camera.xacro (robot description, xacro)
@@ -19,7 +19,8 @@
         <xacro:property name="d435_cam_depth_pz" value="${d435_cam_height/2}"/>
         <!-- Camera position in 3D-->
-        <xacro:property name="d435_cam_x" value="0.370755"/>
+        <xacro:property name="d435_cam_x" value="0.270755"/>
         <xacro:property name="d435_cam_y" value="0.000053"/>
-        <xacro:property name="d435_cam_z" value="0.068583"/>
+        <xacro:property name="d435_cam_z" value="0.010000"/>
+        <!-- <xacro:property name="d435_cam_z" value="0.068583"/> -->
         <!-- <xacro:property name="d435_cam_roll" value="${-M_PI/2}"/> -->
         <xacro:property name="d435_cam_roll" value="0.0"/>
@@ -28,5 +29,5 @@
         <xacro:sensor_d435i parent="${parent}" name="${name}" use_nominal_extrinsics="true">
             <!-- <origin xyz="${0.290755-d435_mesh_x_offset-d435_zero_depth_to_glass - d435_glass_to_front} ${0.000053-d435_cam_depth_pz} ${0.068583}" rpy="${0} 0 0"/> -->
-            <origin xyz="${d435_cam_x-d435_mesh_x_offset-d435_zero_depth_to_glass - d435_glass_to_front} ${0.000053-d435_cam_depth_pz} ${0.068583}" rpy="${d435_cam_roll} 0 0"/>
+            <origin xyz="${d435_cam_x-d435_mesh_x_offset-d435_zero_depth_to_glass - d435_glass_to_front} ${d435_cam_y-d435_cam_depth_pz} ${d435_cam_z}" rpy="${d435_cam_roll} 0 0"/>
         </xacro:sensor_d435i>
         <!-- Link for camera image and gazebe plugin-->

File: robots/go1_description/urdf/go1.urdf (robot description, URDF)
Before this commit: robot go1, 62 links, 61 joints
Joints:
- joint camera_image_joint: origin xyz=0.370755 5.3e-05 0.068583 rpy=0.0 0 0 -> xyz=0.310755 5.3e-05 0.003 rpy=0.0 0 0
- joint d435i_camera_joint: origin xyz=0.35585500000000003 -0.012447000000000001 0.068583 rpy=0.0 0 0 -> xyz=0.29585500000000003 -0.012447000000000001 0.003 rpy=0.0 0 0

File: robots/go1_description/xacro/camera.xacro (robot description, xacro)
@@ -19,7 +19,8 @@
         <xacro:property name="d435_cam_depth_pz" value="${d435_cam_height/2}"/>
         <!-- Camera position in 3D-->
-        <xacro:property name="d435_cam_x" value="0.370755"/>
+        <xacro:property name="d435_cam_x" value="0.310755"/>
         <xacro:property name="d435_cam_y" value="0.000053"/>
-        <xacro:property name="d435_cam_z" value="0.068583"/>
+        <xacro:property name="d435_cam_z" value="0.003000"/>
+        <!-- <xacro:property name="d435_cam_z" value="0.068583"/> -->
         <!-- <xacro:property name="d435_cam_roll" value="${-M_PI/2}"/> -->
         <xacro:property name="d435_cam_roll" value="0.0"/>
@@ -28,5 +29,5 @@
         <xacro:sensor_d435i parent="${parent}" name="${name}" use_nominal_extrinsics="true">
             <!-- <origin xyz="${0.290755-d435_mesh_x_offset-d435_zero_depth_to_glass - d435_glass_to_front} ${0.000053-d435_cam_depth_pz} ${0.068583}" rpy="${0} 0 0"/> -->
-            <origin xyz="${d435_cam_x-d435_mesh_x_offset-d435_zero_depth_to_glass - d435_glass_to_front} ${0.000053-d435_cam_depth_pz} ${0.068583}" rpy="${d435_cam_roll} 0 0"/>
+            <origin xyz="${d435_cam_x-d435_mesh_x_offset-d435_zero_depth_to_glass - d435_glass_to_front} ${d435_cam_y-d435_cam_depth_pz} ${d435_cam_z}" rpy="${d435_cam_roll} 0 0"/>
         </xacro:sensor_d435i>
         <!-- Link for camera image and gazebe plugin-->
